File: TheOpenPursuit/OpenOT/PCB/openot hotswap/openot switchplate/openot rev2.kicad_pcb (KiCad board)
At the start: 2 copper layers, 313.8 x 110.8 mm, 119 parts

Commit message: another openot update
Parts:
- removed the REF** at (291.6, 134.2)
Other:
- outline, holes or cut-outs redrawn
Changed lines of the file:
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@@
     )
-  )
-  (footprint "MountingHole:MountingHole_2.2mm_M2" (layer "F.Cu")
-    (at 291.65 134.25)
-    (descr "Mounting Hole 2.2mm, no annular, M2")
-    (tags "mounting hole 2.2mm no annular m2")
-    (attr exclude_from_pos_files exclude_from_bom)
-    (fp_text reference "REF**" (at 0 -3.2) (layer "F.SilkS")
-      (effects (font (size 1 1) (thickness 0.15)))
-    )
-    (fp_text value "MountingHole_2.2mm_M2" (at 0 3.2) (layer "F.Fab")
-      (effects (font (size 1 1) (thickness 0.15)))
-    )
-    (fp_text user "${REFERENCE}" (at 0.3 0) (layer "F.Fab")
-      (effects (font (size 1 1) (thickness 0.15)))
-    )
-    (fp_circle (center 0 0) (end 2.2 0) (layer "Cmts.User") (width 0.15) (fill none))
-    (fp_circle (center 0 0) (end 2.45 0) (layer "F.CrtYd") (width 0.05) (fill none))
-    (pad "" np_thru_hole circle (at 0 0) (size 2.2 2.2) (drill 2.2) (layers *.Cu *.Mask))
   )
   (footprint "Connector_PinHeader_1.00mm:PinHeader_1x01_P1.00mm_Vertical" (layer "F.Cu")
@@
     (pad "1" smd roundrect locked (at 0 0 180) (size 16 16) (layers "B.Cu" "B.Mask") (roundrect_rratio 0.063))
   )
+  (gr_line (start 364.15 167.5) (end 326.65 167.5) (layer "Edge.Cuts") (width 0.05))
+  (gr_line (start 364.4 129.75) (end 364.15 167.5) (layer "Edge.Cuts") (width 0.05))
   (gr_rect (start 60.995683 77.385634) (end 374.787283 188.180434) (layer "Edge.Cuts") (width 0.1) (fill none))
-  (gr_circle (center 326.9 129.75) (end 325.65 162.5) (layer "Edge.Cuts") (width 0.05) (fill none))
+  (gr_arc (start 326.65 167.5) (mid 299.956719 103.056719) (end 364.4 129.75) (layer "Edge.Cuts") (width 0.05))
   (zone (net 0) (net_name "") (layer "F.Cu") (hatch edge 0.508)
     (connect_pads (clearance 0.508))

Commit message: openot pcb updates
Parts:
- removed the REF** at (85.3, 143.1)
- REF** (x54): value PinHeader_1x01_P1.00mm_Vertical -> empty; footprint Connector_PinHeader_1.00mm:PinHeader_1x01_P1.00mm_Vertical -> keyswitches:empty
- REF**: value MX_FMask-with-cutout -> switchplate cutout stabs; footprint Keebio-Parts:MX_FMask-with-cutout -> Keebio-Parts:switchplate cutout stabs
