File: TheOpenPursuit/OOTstag/OOTstag.kicad_pcb (KiCad board)
At the start: 2 copper layers, 405.8 x 127.2 mm, 301 parts, among them IC1 AP7335-WG-7, J1 Conn_01x06_Female, Q1 DSS60601MZ4-13, SW1 SW_Push, U1 AT90USB1286-AU, U1 XC6206P332MR, U2 PMW3360DM-T2QU, U2 PRTR5V0U2X, U4 TXS0104EDR, Y1 16MHz

Commit message: new pr9oject
Parts:
- added C2: 1uF, Capacitors_SMD:C_0603, B.Cu at (444.0, 186.3)
- added C3: 22pF, Capacitors_SMD:C_0603, B.Cu at (458.3, 195.3)
- added C4: 22pF, Capacitors_SMD:C_0603, B.Cu at (458.3, 191.5)
- added C5: 1uF, Capacitors_SMD:C_0603, B.Cu at (437.4, 189.0)
- added C6: 0.1uF, Capacitors_SMD:C_0603, B.Cu at (436.2, 196.0)
- added C7: 0.1uF, Capacitors_SMD:C_0603, B.Cu at (446.1, 185.6)
- added C8: 0.1uF, Capacitors_SMD:C_0603, B.Cu at (451.3, 189.4)
- added F1: 500mA, Fuse_Holders_and_Fuses:Fuse_SMD1206_Reflow, B.Cu at (435.6, 184.4)
- added J1: AVR-ISP-6, Molex-0548190589:Reset_Pretty-Mask, B.Cu at (473.4, 192.7)
- added RC1: 22, Resistors_SMD:R_0603, B.Cu at (439.0, 183.7)
- added RC2: 22, Resistors_SMD:R_0603, B.Cu at (441.3, 183.7)
- added RC3: 10k, Resistors_SMD:R_0603, B.Cu at (454.5, 188.7)
- added RC4: 1k, Resistors_SMD:R_0603, B.Cu at (442.3, 201.7)
- added RC6: 5k1, Resistors_SMD:R_0603, B.Cu at (436.7, 179.7)
- added RC7: 5k1, Resistors_SMD:R_0603, B.Cu at (443.7, 179.7)
- added SW1: SW_Push, Molex-0548190589:SKQG-1155865, B.Cu at (458.2, 176.3)
- added U1: AT90USB1286-AU, Housings_DFN_QFN:QFN-64-1EP_9x9mm_Pitch0.5mm, B.Cu at (444.1, 193.9)
- added U2: PRTR5V0U2X, locallib:SOT143B, B.Cu at (440.1, 179.7)
- added USB1: HRO-TYPE-C-31-M-12, Type-C:HRO-TYPE-C-31-M-12-Assembly, B.Cu at (440.1, 168.1)
- added Y1: 16MHz, Crystals:Crystal_SMD_3225-4pin_3.2x2.5mm, B.Cu at (454.8, 193.4)
- moved ? 56.3 mm to (446.7, 150.3)
- moved C2 56.3 mm to (462.8, 135.5)
- moved C3 56.3 mm to (448.5, 144.5)
- moved C4 56.3 mm to (448.5, 140.7)
- moved C5 56.3 mm to (469.5, 138.1)
- moved C6 56.3 mm to (470.6, 145.1)
- moved C7 56.3 mm to (460.7, 134.7)
- moved C8 56.3 mm to (455.5, 138.5)
- moved F1 56.3 mm to (471.2, 133.6)
- moved Q1 56.3 mm to (434.7, 141.6)
- moved RC1 56.3 mm to (467.8, 132.8)
- moved RC2 56.3 mm to (465.5, 132.8)
- moved RC3 56.3 mm to (452.3, 137.9)
- moved RC4 56.3 mm to (464.5, 150.8)
- moved RC5 56.3 mm to (441.8, 141.6)
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Routing:
- net (no net): track 287.3 -> 825.2 mm, vias 0 -> 12
- net GND: track 30.9 -> 165.5 mm, vias 6 -> 8
- net MOSI: track 32.1 -> 69.1 mm
- net MISO: track 15.4 -> 48.7 mm
Other:
- board text added: "D16"
- board text added: "D96"
