File: TheOpenPursuit/OOTstag/OOstag rev 2/mykeyboard.kicad_pcb (KiCad board)
At the start: 2 copper layers, 8.5 x 16.7 mm, 213 parts, among them IC1 AP7335-WG-7, J1 Conn_01x06_Female, J1 USB_mini_micro_B, J2 Conn_02x03_Odd_Even, K0 Esc, K1 F1, K10 F10, K11 F11, K12 F12, K13 Home, K14 End, K15 Insert, K16 ~,`, K17 !,1, K18 @,2, K19 #,3, K2 F2, K20 $,4, K21 %,5, K22 ^,6, K23 &,7, K24 *,8, K25 (,9, K26 ),0, K27 _,-, K28 +,=, K29 Backspace, K3 F3, K30 Delete, K31 Tab, K32 Q, K33 W, K34 E, K35 R, K36 T, K37 Y, K38 U, K39 I, K4 F4, K40 O, K41 P, K42 {,[, K43 },], K44 |,\, K45 PgUp, K46 Caps Lock, K47 A, K48 S, K49 D, K5 F5, K50 F, K51 G, K52 H, K53 J, K54 K, K55 L, K56 :,;, K57 ",', K58 Enter, K59 PgDn, K6 F6, K60 Shift, K61 Z, K62 X, K63 C, K64 V, K65 B, K66 N, K67 M, K68 <,,, K69 >,., K7 F7, K70 ?,/, K71 Shift, K72 ↑, K73 Ctrl, K74 Win, K75 Alt, K76 Space, K77 Alt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

Commit message: pcb update
Parts:
- removed the J1 at (335.9, 59.5)
- added REF**: USB_C_Receptacle_GCT_USB4105-xx-A_16P_TopMnt_Horizontal, Connector_USB:USB_C_Receptacle_GCT_USB4105-xx-A_16P_TopMnt_Horizontal, B.Cu at (360.5, 71.0)
- moved C4 28.4 mm to (357.7, 81.5)
- moved R2 28.4 mm to (360.7, 81.6)
- moved R3 28.4 mm to (363.7, 81.6)
- moved H1 23.9 mm to (359.5, 34.5)
- moved H2 23.9 mm to (373.5, 34.5)
- moved H3 23.9 mm to (359.5, 46.5)
- moved H4 23.9 mm to (373.5, 46.5)
Routing:
- net Net-(R3-Pad1): track 12.0 -> 26.0 mm, vias 0 -> 2
- net Net-(R2-Pad1): track 13.4 -> 22.6 mm
- net VCC: track 63.6 -> 70.3 mm
- net Net-(J1-Pad3): track 6.52 -> 7.50 mm
- net Net-(J1-Pad2): track 5.20 -> 6.18 mm

Commit message: pcb trace update
Routing:
- net /Col_1: track 0.00 -> 130.6 mm, vias 0 -> 6
- net /Col_2: track 0.00 -> 121.2 mm, vias 0 -> 6
- net /Col_0: track 0.00 -> 114.3 mm, vias 0 -> 6
- net Net-(D8-Pad2): track 5.23 -> 11.6 mm
- net Net-(D15-Pad2): track 5.23 -> 11.6 mm
- net Net-(D14-Pad2): track 5.23 -> 11.6 mm
- net Net-(D13-Pad2): track 5.23 -> 11.6 mm
- net Net-(D5-Pad2): track 5.23 -> 11.6 mm
- net Net-(D1-Pad2): track 5.23 -> 11.6 mm
- net Net-(D0-Pad2): track 5.23 -> 11.6 mm
- net Net-(D9-Pad2): track 5.23 -> 11.6 mm
- net Net-(D7-Pad2): track 5.23 -> 11.6 mm
- net Net-(D6-Pad2): track 5.23 -> 11.6 mm
- net Net-(D4-Pad2): track 5.23 -> 11.6 mm
- net Net-(D3-Pad2): track 5.23 -> 11.6 mm
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
Commit message: new project update
Parts:
- removed R86 (x4): 1k, Resistors_SMD:R_0603
- D0, D1, D10, D11, D12, D13, D14, D15, D16, D17, D18, D19, D2, D20, D21, D22, D23, D24, D25, D26, D27, D28, D29, D3, D30, D31, D32, D33, D34, D35, D36, D37, D38, D39, D4, D40, D41, D42, D43, D44, D45, D46, D47, D48, D49, D5, D50, D51, D52, D53, D54, D55, D56, D57, D58, D59, D6, D60, D61, D62, D63, D64, D65, D66, D67, D68, D69, D7, D70, D71, D72, D73, D74, D75, D76, D77, D78, D79, D8, D80, D81, D9: footprint Diode_SMD:D_0805_2012Metric_Pad1.15x1.40mm_HandSolder -> Diode_SMD:D_SOD-123
- moved H3 386.0 mm to (3.00, 194.5)
- moved H1 358.5 mm to (2.50, 67.0)
- moved H4 150.4 mm to (403.0, 194.0)
- moved H2 42.9 mm to (401.5, 67.0)
- moved D86 15.9 mm to (362.2, 196.0)
- moved D86 15.9 mm to (382.5, 196.0)
- moved D86 15.9 mm to (323.0, 188.2)
- moved D86 15.9 mm to (342.7, 192.5)
Connections:
- MX_NUM4 pad 1: (no net) -> /Col_9
- MX_NUM5 pad 1: (no net) -> /Col_10
- MX_NUM6 pad 1: (no net) -> /Col_11
- MX_NUM7 pad 1: (no net) -> /Col_12
Routing:
- net /Col_9: track 0.00 -> 222.1 mm, vias 5 -> 6
- net /Col_6: track 0.00 -> 221.6 mm
- net /Col_7: track 0.00 -> 221.1 mm
- net /Col_8: track 0.00 -> 217.8 mm
- net /Col_5: track 0.00 -> 210.5 mm
- net /Col_4: track 0.00 -> 201.3 mm
- net /Col_3: track 0.00 -> 149.1 mm
- net /Col_12: track 0.00 -> 103.8 mm, vias 5 -> 6
- net /Col_11: track 0.00 -> 94.5 mm, vias 5 -> 6
- net /Col_10: track 0.00 -> 91.5 mm, vias 5 -> 6
- net /Col_13: track 0.00 -> 85.5 mm
- net /Col_14: track 0.00 -> 53.1 mm
- net (no net): track 487.1 -> 524.5 mm
- net Net-(D72-Pad2): track 5.23 -> 11.6 mm
- net Net-(D59-Pad2): track 5.23 -> 11.6 mm
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- added copper zone on B.Cu, net GND
- added copper zone on F.Cu, net GND
Other:
- board size 8.5 x 16.7 mm -> 409 x 137 mm

Commit message: rpi pico update
Parts:
- removed the C1 at (326.7, 93.0)
- removed the C2 at (329.7, 79.0)
- removed the C3 at (347.7, 90.0)
- removed the C4 at (357.7, 81.5)
- removed the C5 at (341.7, 79.0)
- removed C6, C7: 22p, Capacitor_SMD:C_0805_2012Metric_Pad1.15x1.40mm_HandSolder
- removed C8: 1u, Capacitor_SMD:C_0805_2012Metric_Pad1.15x1.40mm_HandSolder
- removed J2: Conn_02x03_Odd_Even, Connector_PinHeader_2.54mm:PinHeader_2x03_P2.54mm_Vertical
- removed the R1 at (339.7, 97.0)
- removed the R2 at (360.7, 81.6)
- removed the R3 at (363.7, 81.6)
- removed the R4 at (326.7, 82.0)
- removed the REF** at (402.5, 208.1)
- removed the REF** at (360.5, 71.0)
- removed SW1: SW_Push, Button_Switch_SMD:SW_Push_1P1T_NO_6x6mm_H9.5mm
- removed the U1 at (335.5, 87.8)
- removed Y1: Crystal, Crystal:Crystal_SMD_5032-2Pin_5.0x3.2mm_HandSoldering
- added REF**: RPi_Pico_SMD_TH, MCU_RaspberryPi_and_Boards:RPi_Pico_SMD_TH, F.Cu at (338.2, 88.2)
Connections:
- K15 pad 1: /Col_15 -> /Col_14
Routing:
- net VCC: track 70.3 -> 0.00 mm
- net GND: track 57.5 -> 30.9 mm
- net Net-(R3-Pad1): track 26.0 -> 0.00 mm, vias 2 -> 0
- net /Col_14: track 53.1 -> 78.8 mm, vias 3 -> 4
- net Net-(R2-Pad1): track 22.6 -> 0.00 mm
- net Net-(R1-Pad1): track 22.5 -> 0.00 mm
- net Net-(C7-Pad1): track 15.0 -> 0.00 mm
- net Net-(C6-Pad1): track 14.6 -> 0.00 mm
- net /Row_4: track 259.9 -> 272.8 mm
- net Net-(J1-Pad3): track 7.50 -> 0.00 mm
- net Net-(C8-Pad1): track 6.79 -> 0.00 mm
- net Net-(J1-Pad2): track 6.18 -> 0.00 mm
- net Net-(R4-Pad2): track 11.8 -> 8.11 mm
- net /Col_15: vias 1 -> 0

Commit message: another ootstag update
Parts:
- moved D12 59.3 mm to (297.1, 97.8)
- moved D28 59.3 mm to (297.1, 121.6)
- moved D56 59.3 mm to (273.3, 159.7)
- moved D71 59.3 mm to (309.0, 178.7)
- moved K11 59.3 mm to (283.9, 88.9)
- moved K27 59.3 mm to (283.9, 112.7)
- moved K55 59.3 mm to (260.0, 150.8)
- moved D22 59.3 mm to (182.8, 121.6)
- moved D34 59.3 mm to (135.2, 140.6)
- moved D50 59.3 mm to (159.0, 159.7)
- moved D6 59.3 mm to (182.8, 97.8)
- moved K21 59.3 mm to (169.6, 112.7)
- moved K49 59.3 mm to (145.7, 150.8)
- moved K5 59.3 mm to (169.6, 88.9)
- moved D47 59.3 mm to (101.8, 159.7)
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Connections:
- D15 pad 1: /Row_0 -> /Row_4
- D86 pad 1: (no net) -> /Row_5 (x4)
- REF** pad 1: (no net) -> /Col_0
- REF** pad 10: (no net) -> /Col_7
- REF** pad 11: (no net) -> /Col_8
- REF** pad 12: (no net) -> /Col_9
- REF** pad 14: (no net) -> /Col_10
- REF** pad 15: (no net) -> /Col_11
- REF** pad 16: (no net) -> /Col_12
- REF** pad 17: (no net) -> /Col_13
- REF** pad 19: (no net) -> /Col_14
- REF** pad 2: (no net) -> /Col_1
- REF** pad 4: (no net) -> /Col_2
- REF** pad 5: (no net) -> /Col_3
- REF** pad 6: (no net) -> /Col_4
- REF** pad 7: (no net) -> /Col_5
- REF** pad 9: (no net) -> /Col_6
Routing:
- net (no net): track 524.1 -> 1147.0 mm, vias 8 -> 17
- net /Col_0: track 112.8 -> 422.8 mm, vias 6 -> 7
- net /Col_1: track 129.8 -> 419.2 mm, vias 6 -> 7
- net /Col_2: track 120.8 -> 390.5 mm, vias 6 -> 7
- net /Col_3: track 149.1 -> 400.7 mm, vias 6 -> 7
- net /Col_4: track 201.3 -> 444.9 mm
- net /Row_5: track 288.5 -> 523.9 mm, vias 0 -> 1
- net /Col_5: track 210.5 -> 437.3 mm
- net /Col_6: track 221.6 -> 432.7 mm
- net /Col_7: track 221.1 -> 414.7 mm
- net /Row_4: track 272.8 -> 450.7 mm, vias 0 -> 2
- net /Col_8: track 217.8 -> 393.5 mm
- net /Col_9: track 222.1 -> 381.1 mm
- net /Col_10: track 91.5 -> 233.0 mm, vias 6 -> 5
- net /Col_11: track 94.5 -> 217.5 mm, vias 6 -> 5
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- added copper zone on B.Cu, net (none)
- added copper zone on F.Cu, net (none)
- removed copper zone on B.Cu, net GND
- removed copper zone on F.Cu, net GND
Other:
- board text removed: "15k"
