File: personal 75%/personal 75% final revision/PCB files/switchplate/fr4 plate.kicad_pcb (KiCad board)
At the start: 2 copper layers, 320.1 x 124.8 mm, 0 parts

Commit message: case update
Parts:
- added ?: , , F.Cu at (371.5, 72.6)
- added ?: , , F.Cu at (51.4, 197.5)
- added ?: , , F.Cu at (371.5, 197.5)
- added REF**: MountingHole_6.4mm_M6, MountingHole:MountingHole_6.4mm_M6, F.Cu at (371.5, 72.6)
- added REF**: MountingHole_6.4mm_M6, MountingHole:MountingHole_6.4mm_M6, F.Cu at (371.5, 197.5)
- added REF**: MountingHole_6.4mm_M6, MountingHole:MountingHole_6.4mm_M6, F.Cu at (51.5, 72.6)
- added REF**: MountingHole_6.4mm_M6, MountingHole:MountingHole_6.4mm_M6, F.Cu at (51.4, 197.5)
Changed lines of the file:
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@@
   )
   (net 0 "")
+  (footprint "" (layer "F.Cu")
+    (at 371.494999 72.628)
+    (fp_text reference "" (at 0 0) (layer "F.SilkS")
+      (effects (font (size 1.27 1.27) (thickness 0.15)))
+    )
+    (fp_text value "" (at 0 0) (layer "F.SilkS")
+      (effects (font (size 1.27 1.27) (thickness 0.15)))
+    )
+    (pad "1" thru_hole circle (at 0 0) (size 10.6 10.6) (drill 5.3) (layers F&B.Cu *.Mask))
+  )
+  (footprint "MountingHole:MountingHole_6.4mm_M6" (layer "F.Cu")
+    (at 371.494999 72.628)
+    (descr "Mounting Hole 6.4mm, no annular, M6")
+    (tags "mounting hole 6.4mm no annular m6")
+    (attr exclude_from_pos_files exclude_from_bom)
+    (fp_text reference "REF**" (at 0 -7.4) (layer "F.SilkS")
+      (effects (font (size 1 1) (thickness 0.15)))
+    )
+    (fp_text value "MountingHole_6.4mm_M6" (at 0 7.4) (layer "F.Fab")
+      (effects (font (size 1 1) (thickness 0.15)))
+    )
+    (fp_text user "${REFERENCE}" (at 0 0) (layer "F.Fab")
+      (effects (font (size 1 1) (thickness 0.15)))
+    )
+    (fp_circle (center 0 0) (end 6.4 0) (layer "Cmts.User") (width 0.15) (fill none))
+    (fp_circle (center 0 0) (end 6.65 0) (layer "F.CrtYd") (width 0.05) (fill none))
+    (pad "" np_thru_hole circle (at 0 0) (size 6.4 6.4) (drill 6.4) (layers *.Cu *.Mask))
+  )
+  (footprint "MountingHole:MountingHole_6.4mm_M6" (layer "F.Cu")
+    (at 371.494999 197.458)
+    (descr "Mounting Hole 6.4mm, no annular, M6")
+    (tags "mounting hole 6.4mm no annular m6")
+    (attr exclude_from_pos_files exclude_from_bom)
+    (fp_text reference "REF**" (at 0 -7.4) (layer "F.SilkS")
+      (effects (font (size 1 1) (thickness 0.15)))
+    )
+    (fp_text value "MountingHole_6.4mm_M6" (at 0 7.4) (layer "F.Fab")
+      (effects (font (size 1 1) (thickness 0.15)))
+    )
+    (fp_text user "${REFERENCE}" (at 0 0) (layer "F.Fab")
+      (effects (font (size 1 1) (thickness 0.15)))
+    )
+    (fp_circle (center 0 0) (end 6.4 0) (layer "Cmts.User") (width 0.15) (fill none))
+    (fp_circle (center 0 0) (end 6.65 0) (layer "F.CrtYd") (width 0.05) (fill none))
+    (pad "" np_thru_hole circle (at 0 0) (size 6.4 6.4) (drill 6.4) (layers *.Cu *.Mask))
+  )
+  (footprint "MountingHole:MountingHole_6.4mm_M6" (layer "F.Cu")
+    (at 51.52 72.59)
+    (descr "Mounting Hole 6.4mm, no annular, M6")
+    (tags "mounting hole 6.4mm no annular m6")
+    (attr exclude_from_pos_files exclude_from_bom)
+    (fp_text reference "REF**" (at 0 -7.4) (layer "F.SilkS")
+      (effects (font (size 1 1) (thickness 0.15)))
+    )
+    (fp_text value "MountingHole_6.4mm_M6" (at 0 7.4) (layer "F.Fab")
+      (effects (font (size 1 1) (thickness 0.15)))
+    )
+    (fp_text user "${REFERENCE}" (at 0 0) (layer "F.Fab")
+      (effects (font (size 1 1) (thickness 0.15)))
+    )
+    (fp_circle (center 0 0) (end 6.4 0) (layer "Cmts.User") (width 0.15) (fill none))
+    (fp_circle (center 0 0) (end 6.65 0) (layer "F.CrtYd") (width 0.05) (fill none))
+    (pad "" np_thru_hole circle (at 0 0) (size 6.4 6.4) (drill 6.4) (layers *.Cu *.Mask))
+  )
+  (footprint "" (layer "F.Cu")
+    (at 51.44 197.47)
+    (fp_text reference "" (at 0 0) (layer "F.SilkS")
+      (effects (font (size 1.27 1.27) (thickness 0.15)))
+    )
+    (fp_text value "" (at 0 0) (layer "F.SilkS")
+      (effects (font (size 1.27 1.27) (thickness 0.15)))
+    )
+    (pad "1" thru_hole circle (at 0 0) (size 10.6 10.6) (drill 5.3) (layers F&B.Cu *.Mask))
+  )
+  (footprint "" (layer "F.Cu")
+    (at 371.494999 197.458)
+    (fp_text reference "" (at 0 0) (layer "F.SilkS")
+      (effects (font (size 1.27 1.27) (thickness 0.15)))
+    )
+    (fp_text value "" (at 0 0) (layer "F.SilkS")
+      (effects (font (size 1.27 1.27) (thickness 0.15)))
+    )
+    (pad "1" thru_hole circle (at 0 0) (size 10.6 10.6) (drill 5.3) (layers F&B.Cu *.Mask))
+  )
+  (footprint "MountingHole:MountingHole_6.4mm_M6" (layer "F.Cu")
+    (at 51.44 197.47)
+    (descr "Mounting Hole 6.4mm, no annular, M6")
+    (tags "mounting hole 6.4mm no annular m6")
+    (attr exclude_from_pos_files exclude_from_bom)
+    (fp_text reference "REF**" (at 0 -7.4) (layer "F.SilkS")
+      (effects (font (size 1 1) (thickness 0.15)))
+    )
+    (fp_text value "MountingHole_6.4mm_M6" (at 0 7.4) (layer "F.Fab")
+      (effects (font (size 1 1) (thickness 0.15)))
+    )
+    (fp_text user "${REFERENCE}" (at 0 0) (layer "F.Fab")
+      (effects (font (size 1 1) (thickness 0.15)))
+    )
+    (fp_circle (center 0 0) (end 6.4 0) (layer "Cmts.User") (width 0.15) (fill none))
+    (fp_circle (center 0 0) (end 6.65 0) (layer "F.CrtYd") (width 0.05) (fill none))
+    (pad "" np_thru_hole circle (at 0 0) (size 6.4 6.4) (drill 6.4) (layers *.Cu *.Mask))
+  )
   (gr_line (start 192.281 187.149998) (end 231.906 187.149998) (layer "Edge.Cuts") (width 0.188976))
   (gr_line (start 232.76301 120.700001) (end 232.76301 120.700001) (layer "Edge.Cuts") (width 0.188976))
@@
     (polygon
       (pts
-        (xy 374.794999 63.308)
-        (xy 374.534999 204.768)
-        (xy 45.234999 205.028)
-        (xy 43.944999 63.048)
+        (xy 385.471617 63.327623)
+        (xy 385.211617 204.787623)
+        (xy 42.817715 205.049964)
+        (xy 41.527715 63.069964)
       )
     )
@@
     (polygon
       (pts
-        (xy 374.014999 63.308)
-        (xy 374.534999 204.768)
-        (xy 45.754999 204.508)
-        (xy 44.724999 63.048)
+        (xy 387.687798 63.25774)
+        (xy 388.207798 204.71774)
+        (xy 42.919316 204.528648)
+        (xy 41.889316 63.068648)
       )
     )
