File: New folder/pcb/keyboard.kicad_pcb (KiCad board)
At the start: 2 copper layers, 319.6 x 179.7 mm, 179 parts, among them U1 ATMEGA32U4, X1 XTAL_GND

Commit message: pcb update
Parts:
- added REF**: PinHeader_1x12_P2.54mm_Vertical, Connector_PinHeader_2.54mm:PinHeader_1x12_P2.54mm_Vertical, F.Cu at (262.1, 264.1)
- added REF**: PinHeader_1x12_P2.54mm_Vertical, Connector_PinHeader_2.54mm:PinHeader_1x12_P2.54mm_Vertical, F.Cu at (317.9, 263.9)
- moved C3 207.7 mm to (499.9, 212.5), turned to -90 degrees
- moved C1 203.4 mm to (479.2, 211.7)
- moved C2 203.4 mm to (489.2, 211.7)
- moved C4 203.4 mm to (477.9, 206.0)
- moved C5 203.4 mm to (477.9, 201.0)
- moved C6 203.4 mm to (477.9, 196.0)
- moved C7 203.4 mm to (477.9, 191.0)
- moved REF** 203.4 mm to (482.3, 202.2)
- moved REF** 203.4 mm to (508.7, 185.8)
- moved REF** 203.4 mm to (477.1, 185.8)
- moved U1 203.4 mm to (496.2, 201.1)
- moved X1 203.4 mm to (484.2, 211.7)
- moved R2 203.4 mm to (488.0, 191.2)
- moved R3 202.3 mm to (496.9, 212.5), turned to -90 degrees
- moved R4 195.2 mm to (492.9, 212.5), turned to -90 degrees
Connections:
- REF** pad 1: (no net) -> /col12
- REF** pad 10: (no net) -> /row2
- REF** pad 11: (no net) -> /row1
- REF** pad 12: (no net) -> /row0
- REF** pad 2: (no net) -> /col13
- REF** pad 3: (no net) -> /col14
- REF** pad 4: (no net) -> /col15
- REF** pad 6: (no net) -> /row6
- REF** pad 7: (no net) -> /row5
- REF** pad 8: (no net) -> /row4
- REF** pad 9: (no net) -> /row3
- REF** pad 1: (no net) -> /col0
- REF** pad 10: (no net) -> /col9
- REF** pad 11: (no net) -> /col10
- REF** pad 12: (no net) -> /col11
- REF** pad 2: (no net) -> /col1
- REF** pad 3: (no net) -> /col2
- REF** pad 4: (no net) -> /col3
- REF** pad 5: (no net) -> /col4
- REF** pad 6: (no net) -> /col5
- REF** pad 7: (no net) -> /col6
- REF** pad 8: (no net) -> /col7
- REF** pad 9: (no net) -> /col8
Routing:
- net VCC: track 0.00 -> 63.8 mm
- net Net-(C1-Pad1): track 0.00 -> 30.5 mm, vias 0 -> 2
- net /col0: track 0.00 -> 30.3 mm, vias 0 -> 2
- net /col2: track 0.00 -> 26.6 mm, vias 0 -> 2
- net /col1: track 0.00 -> 25.4 mm, vias 0 -> 1
- net Net-(USB1-Pad2): track 0.00 -> 22.7 mm, vias 0 -> 1
- net Net-(USB1-Pad3): track 0.00 -> 20.8 mm, vias 0 -> 1
- net /col12: track 0.00 -> 20.7 mm, vias 0 -> 1
- net /row2: track 0.00 -> 20.4 mm, vias 0 -> 1
- net /row3: track 0.00 -> 20.2 mm, vias 0 -> 1
- net /col14: track 0.00 -> 19.7 mm, vias 0 -> 1
- net /row4: track 0.00 -> 19.3 mm, vias 0 -> 1
- net /col13: track 0.00 -> 19.0 mm, vias 0 -> 1
- net /col11: track 0.00 -> 18.7 mm
- net /row1: track 0.00 -> 18.5 mm, vias 0 -> 1
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Other:
- board size 319.6 x 179.7 mm -> 370.8 x 133.8 mm
