File: New folder/pcb/main board/_autosave-keyboard.kicad_pcb (KiCad board)
At the start: 2 copper layers, 370.8 x 133.8 mm, 181 parts, among them U1 ATMEGA32U4, X1 XTAL_GND

Commit message: pcb update
Parts:
- added REF**: PinHeader_1x01_P2.54mm_Vertical, Connector_PinHeader_2.54mm:PinHeader_1x01_P2.54mm_Vertical, F.Cu at (429.9, 68.0)
- added REF**: PinHeader_1x02_P2.54mm_Vertical, Connector_PinHeader_2.54mm:PinHeader_1x02_P2.54mm_Vertical, F.Cu at (448.4, 71.8)
- moved REF** 148.9 mm to (420.5, 65.9), turned to 90 degrees
- moved C3 147.7 mm to (447.2, 74.6), turned to 0 degrees
- moved R3 143.8 mm to (447.2, 77.6), turned to 0 degrees
- moved C4 138.7 mm to (443.4, 71.7), turned to 0 degrees
- moved R4 138.7 mm to (447.2, 81.6), turned to 0 degrees
- moved U1 136.8 mm to (435.8, 78.3), turned to 180 degrees
- moved C2 133.4 mm to (446.3, 85.4), turned to 90 degrees
- moved C6 133.0 mm to (428.7, 72.4), turned to 180 degrees
- moved X1 127.1 mm to (446.3, 90.4), turned to -90 degrees
- moved R2 121.8 mm to (425.9, 86.5), turned to -90 degrees
- moved C1 120.8 mm to (446.3, 95.4), turned to 90 degrees
- moved C7 119.6 mm to (427.7, 82.5), turned to -135 degrees
- moved REF** 118.9 mm to (436.9, 92.3), turned to -90 degrees
- moved C5 115.3 mm to (439.9, 92.2), turned to 0 degrees
- moved REF** 104.9 mm to (420.5, 97.5), turned to 180 degrees
Connections:
- REF** pad 5: (no net) -> Net-(U1-Pad43)
- U1 pad 34: Net-(U1-Pad34) -> VCC
- U1 pad 36: Net-(U1-Pad36) -> Net-(U1-Pad43)
- U1 pad 43: Net-(U1-Pad43) -> GND
Routing:
- net (no net): track 0.00 -> 46.1 mm, vias 0 -> 4
- net VCC: track 63.8 -> 50.9 mm, vias 0 -> 2
- net Net-(U1-Pad42): track 0.00 -> 10.9 mm
- net Net-(C1-Pad1): track 30.5 -> 21.3 mm
- net Net-(U1-Pad43): track 0.00 -> 7.46 mm, vias 0 -> 2
- net Net-(C2-Pad1): track 8.60 -> 15.9 mm, vias 0 -> 2
- net Net-(USB1-Pad2): track 22.7 -> 21.5 mm
Other:
- board size 370.8 x 133.8 mm -> 319.6 x 213.7 mm
