File: New folder/pcb/main board/keyboard.kicad_pcb (KiCad board)
At the start: 2 copper layers, 371.4 x 133.8 mm, 183 parts, among them U1 ATMEGA32U4, X1 XTAL_GND

Commit message: pcb update
Parts:
- removed C1, C2, C3, C4, C5, C6, C7: 22pF, Capacitor_SMD:C_0805_2012Metric_Pad1.15x1.40mm_HandSolder
- removed R2: 10k, Resistor_SMD:R_0805_2012Metric_Pad1.15x1.40mm_HandSolder
- removed R3, R4: 22, Resistor_SMD:R_0805_2012Metric_Pad1.15x1.40mm_HandSolder
- removed the REF** at (497.9, 213.0)
- removed the REF** at (490.9, 188.8)
- removed the REF** at (509.4, 192.5)
- removed the REF** at (481.5, 186.6)
- removed the REF** at (481.5, 218.2)
- removed U1: ATMEGA32U4, Package_QFP:TQFP-44_10x10mm_P0.8mm
- removed X1: XTAL_GND, Crystal:Crystal_SMD_5032-4Pin_5.0x3.2mm
- D_0, D_1, D_10, D_11, D_12, D_13, D_14, D_15, D_16, D_17, D_18, D_19, D_2, D_20, D_21, D_22, D_23, D_24, D_25, D_26, D_28, D_29, D_3, D_30, D_31, D_32, D_33, D_34, D_35, D_36, D_37, D_38, D_39, D_4, D_40, D_41, D_42, D_43, D_44, D_45, D_46, D_47, D_48, D_49, D_5, D_50, D_51, D_52, D_53, D_54, D_55, D_56, D_57, D_58, D_59, D_6, D_60, D_61, D_62, D_63, D_64, D_65, D_66, D_67, D_68, D_69, D_7, D_71, D_73, D_74, D_75, D_76, D_77, D_78, D_79, D_8, D_9, D_SPACE, D_SPACE2, D_SPACE3, D_SPACE4: footprint keyboard_parts:D_SOD123_axial -> MX_ALPS_Hybrid:nothing
- K_0, K_1, K_10, K_11, K_12, K_13, K_14, K_15, K_16, K_17, K_18, K_19, K_2, K_20, K_21, K_22, K_23, K_24, K_25, K_28, K_29, K_3, K_30, K_31, K_32, K_33, K_34, K_35, K_36, K_37, K_38, K_39, K_4, K_40, K_41, K_42, K_43, K_44, K_45, K_46, K_47, K_48, K_49, K_5, K_50, K_51, K_52, K_53, K_54, K_56, K_58, K_59, K_6, K_60, K_61, K_62, K_63, K_64, K_65, K_66, K_67, K_68, K_69, K_7, K_71, K_73, K_75, K_76, K_77, K_78, K_79, K_8, K_9, K_SPACE, K_SPACE2, K_SPACE3, K_SPACE4: footprint keyswitches:Kailh_socket_MX -> MX_ALPS_Hybrid:hotswap mx wdiode
- REF**: value Kailh_socket_MX -> hotswap mx wdiode; footprint keyswitches:Kailh_socket_MX -> MX_ALPS_Hybrid:hotswap mx wdiode
- moved REF** 82.1 mm to (235.8, 264.4), turned to 90 degrees
- moved REF** 54.3 mm to (316.4, 264.4)
Connections:
- K_0 pad 1: /col0 -> (no net)
- K_0 pad 2: Net-(D_0-Pad2) -> (no net)
- K_1 pad 1: /col1 -> (no net)
- K_1 pad 2: Net-(D_1-Pad2) -> (no net)
- K_10 pad 1: /col11 -> (no net)
- K_10 pad 2: Net-(D_10-Pad2) -> (no net)
- K_11 pad 1: /col12 -> (no net)
- K_11 pad 2: Net-(D_11-Pad2) -> (no net)
- K_12 pad 1: /col13 -> (no net)
- K_12 pad 2: Net-(D_12-Pad2) -> (no net)
- K_13 pad 1: /col0 -> (no net)
- K_13 pad 2: Net-(D_13-Pad2) -> (no net)
- K_14 pad 1: /col1 -> (no net)
- K_14 pad 2: Net-(D_14-Pad2) -> (no net)
- K_15 pad 1: /col2 -> (no net)
- K_15 pad 2: Net-(D_15-Pad2) -> (no net)
- K_16 pad 1: /col3 -> (no net)
- K_16 pad 2: Net-(D_16-Pad2) -> (no net)
- K_17 pad 1: /col4 -> (no net)
- K_17 pad 2: Net-(D_17-Pad2) -> (no net)
- K_18 pad 1: /col5 -> (no net)
- K_18 pad 2: Net-(D_18-Pad2) -> (no net)
- K_19 pad 1: /col6 -> (no net)
- K_19 pad 2: Net-(D_19-Pad2) -> (no net)
- K_2 pad 1: /col2 -> (no net)
- K_2 pad 2: Net-(D_2-Pad2) -> (no net)
- K_20 pad 1: /col7 -> (no net)
- K_20 pad 2: Net-(D_20-Pad2) -> (no net)
- K_21 pad 1: /col8 -> (no net)
- K_21 pad 2: Net-(D_21-Pad2) -> (no net)
- K_22 pad 1: /col9 -> (no net)
- K_22 pad 2: Net-(D_22-Pad2) -> (no net)
- K_23 pad 1: /col10 -> (no net)
- K_23 pad 2: Net-(D_23-Pad2) -> (no net)
- K_24 pad 1: /col11 -> (no net)
- K_24 pad 2: Net-(D_24-Pad2) -> (no net)
- K_25 pad 1: /col12 -> (no net)
- K_25 pad 2: Net-(D_25-Pad2) -> (no net)
- K_26 pad 1: /col14 -> (no net)
- K_26 pad 2: Net-(D_26-Pad2) -> (no net)
- K_28 pad 1: /col0 -> (no net)
- K_28 pad 2: Net-(D_28-Pad2) -> (no net)
- K_29 pad 1: /col2 -> (no net)
- K_29 pad 2: Net-(D_29-Pad2) -> (no net)
- K_3 pad 1: /col3 -> (no net)
- K_3 pad 2: Net-(D_3-Pad2) -> (no net)
- K_30 pad 1: /col3 -> (no net)
- K_30 pad 2: Net-(D_30-Pad2) -> (no net)
- K_31 pad 1: /col4 -> (no net)
- K_31 pad 2: Net-(D_31-Pad2) -> (no net)
- K_32 pad 1: /col5 -> (no net)
- K_32 pad 2: Net-(D_32-Pad2) -> (no net)
- K_33 pad 1: /col6 -> (no net)
- K_33 pad 2: Net-(D_33-Pad2) -> (no net)
- K_34 pad 1: /col7 -> (no net)
- K_34 pad 2: Net-(D_34-Pad2) -> (no net)
- K_35 pad 1: /col8 -> (no net)
- K_35 pad 2: Net-(D_35-Pad2) -> (no net)
- K_36 pad 1: /col9 -> (no net)
- K_36 pad 2: Net-(D_36-Pad2) -> (no net)
- K_37 pad 1: /col10 -> (no net)
- K_37 pad 2: Net-(D_37-Pad2) -> (no net)
- K_38 pad 1: /col11 -> (no net)
- K_38 pad 2: Net-(D_38-Pad2) -> (no net)
- K_39 pad 1: /col12 -> (no net)
- K_39 pad 2: Net-(D_39-Pad2) -> (no net)
- K_4 pad 1: /col4 -> (no net)
- K_4 pad 2: Net-(D_4-Pad2) -> (no net)
- K_40 pad 1: /col13 -> (no net)
- K_40 pad 2: Net-(D_40-Pad2) -> (no net)
- K_41 pad 1: /col14 -> (no net)
- K_41 pad 2: Net-(D_41-Pad2) -> (no net)
- K_42 pad 1: /col15 -> (no net)
- K_42 pad 2: Net-(D_42-Pad2) -> (no net)
- K_43 pad 1: /col0 -> (no net)
- K_43 pad 2: Net-(D_43-Pad2) -> (no net)
- K_44 pad 1: /col2 -> (no net)
- K_44 pad 2: Net-(D_44-Pad2) -> (no net)
- K_45 pad 1: /col3 -> (no net)
- K_45 pad 2: Net-(D_45-Pad2) -> (no net)
- K_46 pad 1: /col4 -> (no net)
- K_46 pad 2: Net-(D_46-Pad2) -> (no net)
- K_47 pad 1: /col5 -> (no net)
- K_47 pad 2: Net-(D_47-Pad2) -> (no net)
- K_48 pad 1: /col6 -> (no net)
- K_48 pad 2: Net-(D_48-Pad2) -> (no net)
- K_49 pad 1: /col7 -> (no net)
- K_49 pad 2: Net-(D_49-Pad2) -> (no net)
- K_5 pad 1: /col6 -> (no net)
- K_5 pad 2: Net-(D_5-Pad2) -> (no net)
- K_50 pad 1: /col8 -> (no net)
- K_50 pad 2: Net-(D_50-Pad2) -> (no net)
- K_51 pad 1: /col9 -> (no net)
- K_51 pad 2: Net-(D_51-Pad2) -> (no net)
- K_52 pad 1: /col10 -> (no net)
- K_52 pad 2: Net-(D_52-Pad2) -> (no net)
- K_53 pad 1: /col11 -> (no net)
- K_53 pad 2: Net-(D_53-Pad2) -> (no net)
- K_54 pad 1: /col12 -> (no net)
- K_54 pad 2: Net-(D_54-Pad2) -> (no net)
- K_55 pad 1: /col13 -> (no net)
- K_55 pad 2: Net-(D_55-Pad2) -> (no net)
- K_56 pad 1: /col15 -> (no net)
- K_56 pad 2: Net-(D_56-Pad2) -> (no net)
- K_57 pad 1: /col1 -> (no net)
- K_57 pad 2: Net-(D_57-Pad2) -> (no net)
- K_58 pad 1: /col2 -> (no net)
- K_58 pad 2: Net-(D_58-Pad2) -> (no net)
- K_59 pad 1: /col3 -> (no net)
- K_59 pad 2: Net-(D_59-Pad2) -> (no net)
- K_6 pad 1: /col7 -> (no net)
- K_6 pad 2: Net-(D_6-Pad2) -> (no net)
- K_60 pad 1: /col4 -> (no net)
- K_60 pad 2: Net-(D_60-Pad2) -> (no net)
- K_61 pad 1: /col5 -> (no net)
- K_61 pad 2: Net-(D_61-Pad2) -> (no net)
- K_62 pad 1: /col6 -> (no net)
- K_62 pad 2: Net-(D_62-Pad2) -> (no net)
- K_63 pad 1: /col7 -> (no net)
- K_63 pad 2: Net-(D_63-Pad2) -> (no net)
- K_64 pad 1: /col8 -> (no net)
- K_64 pad 2: Net-(D_64-Pad2) -> (no net)
- K_65 pad 1: /col9 -> (no net)
- K_65 pad 2: Net-(D_65-Pad2) -> (no net)
- K_66 pad 1: /col10 -> (no net)
- K_66 pad 2: Net-(D_66-Pad2) -> (no net)
- K_67 pad 1: /col11 -> (no net)
- K_67 pad 2: Net-(D_67-Pad2) -> (no net)
- K_68 pad 1: /col13 -> (no net)
- K_68 pad 2: Net-(D_68-Pad2) -> (no net)
- K_69 pad 1: /col14 -> (no net)
- K_69 pad 2: Net-(D_69-Pad2) -> (no net)
- K_7 pad 1: /col8 -> (no net)
- K_7 pad 2: Net-(D_7-Pad2) -> (no net)
- K_71 pad 1: /col0 -> (no net)
- K_71 pad 2: Net-(D_71-Pad2) -> (no net)
- K_73 pad 1: /col3 -> (no net)
- K_73 pad 2: Net-(D_73-Pad2) -> (no net)
- K_75 pad 1: /col10 -> (no net)
- K_75 pad 2: Net-(D_75-Pad2) -> (no net)
- K_76 pad 1: /col12 -> (no net)
- K_76 pad 2: Net-(D_76-Pad2) -> (no net)
- K_77 pad 1: /col13 -> (no net)
- K_77 pad 2: Net-(D_77-Pad2) -> (no net)
- K_78 pad 1: /col14 -> (no net)
- K_78 pad 2: Net-(D_78-Pad2) -> (no net)
- K_79 pad 1: /col15 -> (no net)
- K_79 pad 2: Net-(D_79-Pad2) -> (no net)
- K_8 pad 1: /col9 -> (no net)
- K_8 pad 2: Net-(D_8-Pad2) -> (no net)
- K_9 pad 1: /col10 -> (no net)
- K_9 pad 2: Net-(D_9-Pad2) -> (no net)
- K_SPACE pad 1: /col14 -> (no net)
- K_SPACE pad 2: Net-(D_SPACE-Pad2) -> (no net)
- K_SPACE2 pad 1: /col15 -> (no net)
- K_SPACE2 pad 2: Net-(D_SPACE2-Pad2) -> (no net)
- K_SPACE3 pad 1: /col1 -> (no net)
- K_SPACE3 pad 2: Net-(D_SPACE3-Pad2) -> (no net)
- K_SPACE4 pad 1: /col11 -> (no net)
- K_SPACE4 pad 2: Net-(D_SPACE4-Pad2) -> (no net)
Routing:
- net (no net): track 46.1 -> 3383.0 mm, vias 4 -> 0
- net VCC: track 69.4 -> 0.00 mm, vias 2 -> 0
- net /col0: track 30.3 -> 0.00 mm, vias 2 -> 0
- net /col2: track 26.6 -> 0.00 mm, vias 2 -> 0
- net /col1: track 25.4 -> 0.00 mm, vias 1 -> 0
- net Net-(USB1-Pad2): track 21.5 -> 0.00 mm, vias 1 -> 0
- net Net-(C1-Pad1): track 21.3 -> 0.00 mm, vias 2 -> 0
- net Net-(USB1-Pad3): track 20.8 -> 0.00 mm, vias 1 -> 0
- net /col12: track 20.7 -> 0.00 mm, vias 1 -> 0
- net /row2: track 20.4 -> 0.00 mm, vias 1 -> 0
- net /row3: track 20.2 -> 0.00 mm, vias 1 -> 0
- net /col14: track 19.7 -> 0.00 mm, vias 1 -> 0
- net /row4: track 19.3 -> 0.00 mm, vias 1 -> 0
- net /col13: track 19.0 -> 0.00 mm, vias 1 -> 0
- net /col11: track 18.7 -> 0.00 mm
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- added copper zone on B.Cu, net (none)
- added copper zone on F.Cu, net (none)
- removed copper zone on B.Cu, net GND
- removed copper zone on F.Cu, net VCC
Other:
- board size 371.4 x 133.8 mm -> 319.6 x 133.8 mm
- board text removed: "PCB Builder by MisterKeebs - mrkeebs.com"
