File: New folder1 - Copy/pcb/main board/_autosave-keyboard.kicad_pcb (KiCad board)
At the start: 2 copper layers, 319.6 x 213.7 mm, 183 parts, among them U1 ATMEGA32U4, X1 XTAL_GND

Commit message: second copy made
Parts:
- removed C1, C2, C3, C4, C5, C6, C7: 22pF, Capacitor_SMD:C_0805_2012Metric_Pad1.15x1.40mm_HandSolder
- removed R2: 10k, Resistor_SMD:R_0805_2012Metric_Pad1.15x1.40mm_HandSolder
- removed R3, R4: 22, Resistor_SMD:R_0805_2012Metric_Pad1.15x1.40mm_HandSolder
- removed the REF** at (436.9, 92.3)
- removed the REF** at (429.9, 68.0)
- removed the REF** at (448.4, 71.8)
- removed the REF** at (420.5, 65.9)
- removed the REF** at (420.5, 97.5)
- removed U1: ATMEGA32U4, Package_QFP:TQFP-44_10x10mm_P0.8mm
- removed X1: XTAL_GND, Crystal:Crystal_SMD_5032-4Pin_5.0x3.2mm
- D_0, D_1, D_10, D_11, D_12, D_13, D_14, D_15, D_16, D_17, D_18, D_19, D_2, D_20, D_21, D_22, D_23, D_24, D_25, D_26, D_28, D_29, D_3, D_30, D_31, D_32, D_33, D_34, D_35, D_36, D_37, D_38, D_39, D_4, D_40, D_41, D_42, D_43, D_44, D_45, D_46, D_47, D_48, D_49, D_5, D_50, D_51, D_52, D_53, D_54, D_55, D_56, D_57, D_58, D_59, D_6, D_60, D_61, D_62, D_63, D_64, D_65, D_66, D_67, D_68, D_69, D_7, D_71, D_73, D_74, D_75, D_76, D_77, D_78, D_79, D_8, D_9, D_SPACE, D_SPACE2, D_SPACE3, D_SPACE4: footprint keyboard_parts:D_SOD123_axial -> keyboard_parts:nothing
- K_0, K_1, K_10, K_11, K_12, K_13, K_14, K_15, K_16, K_17, K_18, K_19, K_2, K_20, K_21, K_22, K_23, K_24, K_25, K_28, K_29, K_3, K_30, K_31, K_32, K_33, K_34, K_35, K_36, K_37, K_38, K_39, K_4, K_40, K_41, K_42, K_43, K_44, K_45, K_46, K_47, K_48, K_49, K_5, K_50, K_51, K_52, K_53, K_54, K_56, K_58, K_59, K_6, K_60, K_61, K_62, K_63, K_64, K_65, K_66, K_67, K_68, K_69, K_7, K_71, K_73, K_75, K_76, K_77, K_78, K_79, K_8, K_9, K_SPACE, K_SPACE2, K_SPACE3, K_SPACE4: footprint keyswitches:Kailh_socket_MX -> MX_ALPS_Hybrid:hotswap with diode
- REF**: value Kailh_socket_MX -> hotswap with diode; footprint keyswitches:Kailh_socket_MX -> MX_ALPS_Hybrid:hotswap with diode
Routing:
- net VCC: track 50.9 -> 0.00 mm, vias 2 -> 0
- net (no net): track 46.1 -> 0.00 mm, vias 4 -> 0
- net /col0: track 30.3 -> 0.00 mm, vias 2 -> 0
- net /col2: track 26.6 -> 0.00 mm, vias 2 -> 0
- net /col1: track 25.4 -> 0.00 mm, vias 1 -> 0
- net Net-(USB1-Pad2): track 21.5 -> 0.00 mm, vias 1 -> 0
- net Net-(C1-Pad1): track 21.3 -> 0.00 mm, vias 2 -> 0
- net Net-(USB1-Pad3): track 20.8 -> 0.00 mm, vias 1 -> 0
- net /col12: track 20.7 -> 0.00 mm, vias 1 -> 0
- net /row2: track 20.4 -> 0.00 mm, vias 1 -> 0
- net /row3: track 20.2 -> 0.00 mm, vias 1 -> 0
- net /col14: track 19.7 -> 0.00 mm, vias 1 -> 0
- net /row4: track 19.3 -> 0.00 mm, vias 1 -> 0
- net /col13: track 19.0 -> 0.00 mm, vias 1 -> 0
- net /col11: track 18.7 -> 0.00 mm
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Other:
- board size 319.6 x 213.7 mm -> 319.6 x 133.8 mm
- board text removed: "PCB Builder by MisterKeebs - mrkeebs.com"
