File: New folder1 - Copy/pcb/mcu daughterboard/mcu daughterboard.kicad_pcb (KiCad board)
At the start: 2 copper layers, 32.2 x 36.7 mm, 17 parts, among them U1 ATMEGA32U4, X1 XTAL_GND

Commit message: second copy made
Parts:
- added REF**: MountingHole_2.2mm_M2_DIN965, MountingHole:MountingHole_2.2mm_M2_DIN965, F.Cu at (147.9, 118.2)
Other:
- outline, holes or cut-outs redrawn
