File: New folder/pcb/mcu daughterboard/mcu daughterboard.kicad_pcb (KiCad board)
At the start: 2 copper layers, 32.2 x 36.7 mm, 17 parts, among them U1 ATMEGA32U4, X1 XTAL_GND

Commit message: graphic added
Parts:
- moved C4 138.9 mm to (148.3, 90.0)
- moved C6 138.2 mm to (131.9, 93.0)
- moved * 136.9 mm to (135.0, 88.7)
- moved * 136.9 mm to (125.6, 86.5)
- moved C1 136.9 mm to (151.4, 116.0)
- moved C2 136.9 mm to (154.0, 105.5)
- moved C3 136.9 mm to (152.3, 95.3)
- moved C7 136.9 mm to (130.3, 117.1)
- moved R2 136.9 mm to (131.0, 107.2)
- moved R3 136.9 mm to (152.3, 98.3)
- moved R4 136.9 mm to (152.3, 102.3)
- moved U1 136.9 mm to (140.9, 99.0)
- moved X1 136.9 mm to (151.4, 111.0)
- moved * 136.9 mm to (142.0, 112.9)
- moved * 136.9 mm to (153.5, 92.4)
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Routing:
- net VCC: track 64.6 -> 69.7 mm

Commit message: pcb update
Other:
- outline, holes or cut-outs redrawn
- board text added: "Reset"
- board text added: "^encoder"
- board text added: "|<-----C0-C11---->|"
- board text added: "|<-R0-R6->|"
- board text added: "|C12-C15|"
