File: 75% rev2/pcb/main board/_autosave-keyboard.kicad_pcb (KiCad board)
At the start: 2 copper layers, 319.6 x 133.8 mm, 166 parts

Commit message: pcb file update
Connections:
- K_0 pad 1: /col0 -> (no net)
- K_0 pad 2: Net-(D_0-Pad2) -> (no net)
- K_1 pad 1: /col1 -> (no net)
- K_1 pad 2: Net-(D_1-Pad2) -> (no net)
- K_10 pad 1: /col11 -> (no net)
- K_10 pad 2: Net-(D_10-Pad2) -> (no net)
- K_11 pad 1: /col12 -> (no net)
- K_11 pad 2: Net-(D_11-Pad2) -> (no net)
- K_12 pad 1: /col13 -> (no net)
- K_12 pad 2: Net-(D_12-Pad2) -> (no net)
- K_13 pad 1: /col0 -> (no net)
- K_13 pad 2: Net-(D_13-Pad2) -> (no net)
- K_14 pad 1: /col1 -> (no net)
- K_14 pad 2: Net-(D_14-Pad2) -> (no net)
- K_15 pad 1: /col2 -> (no net)
- K_15 pad 2: Net-(D_15-Pad2) -> (no net)
- K_16 pad 1: /col3 -> (no net)
- K_16 pad 2: Net-(D_16-Pad2) -> (no net)
- K_17 pad 1: /col4 -> (no net)
- K_17 pad 2: Net-(D_17-Pad2) -> (no net)
- K_18 pad 1: /col5 -> (no net)
- K_18 pad 2: Net-(D_18-Pad2) -> (no net)
- K_19 pad 1: /col6 -> (no net)
- K_19 pad 2: Net-(D_19-Pad2) -> (no net)
- K_2 pad 1: /col2 -> (no net)
- K_2 pad 2: Net-(D_2-Pad2) -> (no net)
- K_20 pad 1: /col7 -> (no net)
- K_20 pad 2: Net-(D_20-Pad2) -> (no net)
- K_21 pad 1: /col8 -> (no net)
- K_21 pad 2: Net-(D_21-Pad2) -> (no net)
- K_22 pad 1: /col9 -> (no net)
- K_22 pad 2: Net-(D_22-Pad2) -> (no net)
- K_23 pad 1: /col10 -> (no net)
- K_23 pad 2: Net-(D_23-Pad2) -> (no net)
- K_24 pad 1: /col11 -> (no net)
- K_24 pad 2: Net-(D_24-Pad2) -> (no net)
- K_25 pad 1: /col12 -> (no net)
- K_25 pad 2: Net-(D_25-Pad2) -> (no net)
- K_26 pad 1: /col14 -> (no net)
- K_26 pad 2: Net-(D_26-Pad2) -> (no net)
- K_28 pad 1: /col0 -> (no net)
- K_28 pad 2: Net-(D_28-Pad2) -> (no net)
- K_29 pad 1: /col2 -> (no net)
- K_29 pad 2: Net-(D_29-Pad2) -> (no net)
- K_3 pad 1: /col3 -> (no net)
- K_3 pad 2: Net-(D_3-Pad2) -> (no net)
- K_30 pad 1: /col3 -> (no net)
- K_30 pad 2: Net-(D_30-Pad2) -> (no net)
- K_31 pad 1: /col4 -> (no net)
- K_31 pad 2: Net-(D_31-Pad2) -> (no net)
- K_32 pad 1: /col5 -> (no net)
- K_32 pad 2: Net-(D_32-Pad2) -> (no net)
- K_33 pad 1: /col6 -> (no net)
- K_33 pad 2: Net-(D_33-Pad2) -> (no net)
- K_34 pad 1: /col7 -> (no net)
- K_34 pad 2: Net-(D_34-Pad2) -> (no net)
- K_35 pad 1: /col8 -> (no net)
- K_35 pad 2: Net-(D_35-Pad2) -> (no net)
- K_36 pad 1: /col9 -> (no net)
- K_36 pad 2: Net-(D_36-Pad2) -> (no net)
- K_37 pad 1: /col10 -> (no net)
- K_37 pad 2: Net-(D_37-Pad2) -> (no net)
- K_38 pad 1: /col11 -> (no net)
- K_38 pad 2: Net-(D_38-Pad2) -> (no net)
- K_39 pad 1: /col12 -> (no net)
- K_39 pad 2: Net-(D_39-Pad2) -> (no net)
- K_4 pad 1: /col4 -> (no net)
- K_4 pad 2: Net-(D_4-Pad2) -> (no net)
- K_40 pad 1: /col13 -> (no net)
- K_40 pad 2: Net-(D_40-Pad2) -> (no net)
- K_41 pad 1: /col14 -> (no net)
- K_41 pad 2: Net-(D_41-Pad2) -> (no net)
- K_42 pad 1: /col15 -> (no net)
- K_42 pad 2: Net-(D_42-Pad2) -> (no net)
- K_43 pad 1: /col0 -> (no net)
- K_43 pad 2: Net-(D_43-Pad2) -> (no net)
- K_44 pad 1: /col2 -> (no net)
- K_44 pad 2: Net-(D_44-Pad2) -> (no net)
- K_45 pad 1: /col3 -> (no net)
- K_45 pad 2: Net-(D_45-Pad2) -> (no net)
- K_46 pad 1: /col4 -> (no net)
- K_46 pad 2: Net-(D_46-Pad2) -> (no net)
- K_47 pad 1: /col5 -> (no net)
- K_47 pad 2: Net-(D_47-Pad2) -> (no net)
- K_48 pad 1: /col6 -> (no net)
- K_48 pad 2: Net-(D_48-Pad2) -> (no net)
- K_49 pad 1: /col7 -> (no net)
- K_49 pad 2: Net-(D_49-Pad2) -> (no net)
- K_5 pad 1: /col6 -> (no net)
- K_5 pad 2: Net-(D_5-Pad2) -> (no net)
- K_50 pad 1: /col8 -> (no net)
- K_50 pad 2: Net-(D_50-Pad2) -> (no net)
- K_51 pad 1: /col9 -> (no net)
- K_51 pad 2: Net-(D_51-Pad2) -> (no net)
- K_52 pad 1: /col10 -> (no net)
- K_52 pad 2: Net-(D_52-Pad2) -> (no net)
- K_53 pad 1: /col11 -> (no net)
- K_53 pad 2: Net-(D_53-Pad2) -> (no net)
- K_54 pad 1: /col12 -> (no net)
- K_54 pad 2: Net-(D_54-Pad2) -> (no net)
- K_55 pad 1: /col13 -> (no net)
- K_55 pad 2: Net-(D_55-Pad2) -> (no net)
- K_56 pad 1: /col15 -> (no net)
- K_56 pad 2: Net-(D_56-Pad2) -> (no net)
- K_57 pad 1: /col1 -> (no net)
- K_57 pad 2: Net-(D_57-Pad2) -> (no net)
- K_58 pad 1: /col2 -> (no net)
- K_58 pad 2: Net-(D_58-Pad2) -> (no net)
- K_59 pad 1: /col3 -> (no net)
- K_59 pad 2: Net-(D_59-Pad2) -> (no net)
- K_6 pad 1: /col7 -> (no net)
- K_6 pad 2: Net-(D_6-Pad2) -> (no net)
- K_60 pad 1: /col4 -> (no net)
- K_60 pad 2: Net-(D_60-Pad2) -> (no net)
- K_61 pad 1: /col5 -> (no net)
- K_61 pad 2: Net-(D_61-Pad2) -> (no net)
- K_62 pad 1: /col6 -> (no net)
- K_62 pad 2: Net-(D_62-Pad2) -> (no net)
- K_63 pad 1: /col7 -> (no net)
- K_63 pad 2: Net-(D_63-Pad2) -> (no net)
- K_64 pad 1: /col8 -> (no net)
- K_64 pad 2: Net-(D_64-Pad2) -> (no net)
- K_65 pad 1: /col9 -> (no net)
- K_65 pad 2: Net-(D_65-Pad2) -> (no net)
- K_66 pad 1: /col10 -> (no net)
- K_66 pad 2: Net-(D_66-Pad2) -> (no net)
- K_67 pad 1: /col11 -> (no net)
- K_67 pad 2: Net-(D_67-Pad2) -> (no net)
- K_68 pad 1: /col13 -> (no net)
- K_68 pad 2: Net-(D_68-Pad2) -> (no net)
- K_69 pad 1: /col14 -> (no net)
- K_69 pad 2: Net-(D_69-Pad2) -> (no net)
- K_7 pad 1: /col8 -> (no net)
- K_7 pad 2: Net-(D_7-Pad2) -> (no net)
- K_71 pad 1: /col0 -> (no net)
- K_71 pad 2: Net-(D_71-Pad2) -> (no net)
- K_73 pad 1: /col3 -> (no net)
- K_73 pad 2: Net-(D_73-Pad2) -> (no net)
- K_75 pad 1: /col10 -> (no net)
- K_75 pad 2: Net-(D_75-Pad2) -> (no net)
- K_76 pad 1: /col12 -> (no net)
- K_76 pad 2: Net-(D_76-Pad2) -> (no net)
- K_77 pad 1: /col13 -> (no net)
- K_77 pad 2: Net-(D_77-Pad2) -> (no net)
- K_78 pad 1: /col14 -> (no net)
- K_78 pad 2: Net-(D_78-Pad2) -> (no net)
- K_79 pad 1: /col15 -> (no net)
- K_79 pad 2: Net-(D_79-Pad2) -> (no net)
- K_8 pad 1: /col9 -> (no net)
- K_8 pad 2: Net-(D_8-Pad2) -> (no net)
- K_9 pad 1: /col10 -> (no net)
- K_9 pad 2: Net-(D_9-Pad2) -> (no net)
- K_SPACE pad 1: /col14 -> (no net)
- K_SPACE pad 2: Net-(D_SPACE-Pad2) -> (no net)
- K_SPACE2 pad 1: /col15 -> (no net)
- K_SPACE2 pad 2: Net-(D_SPACE2-Pad2) -> (no net)
- K_SPACE3 pad 1: /col1 -> (no net)
- K_SPACE3 pad 2: Net-(D_SPACE3-Pad2) -> (no net)
- K_SPACE4 pad 1: /col11 -> (no net)
- K_SPACE4 pad 2: Net-(D_SPACE4-Pad2) -> (no net)
Routing:
- net (no net): track 0.00 -> 4735.3 mm, vias 0 -> 8
- added copper zone on B.Cu, net (none)
- added copper zone on F.Cu, net (none)
- removed copper zone on B.Cu, net GND
- removed copper zone on F.Cu, net VCC

Commit message: updates
Parts:
- removed K_68: KEYSW, MX_ALPS_Hybrid:hotswap with diode
- added D**: D, keyboard_parts:D_SOD123_axial, B.Cu at (387.3, 242.3)
- added D**: D, keyboard_parts:D_SOD123_axial, B.Cu at (404.2, 184.9)
- added D**: D, keyboard_parts:D_SOD123_axial, B.Cu at (158.7, 242.4)
- added D**: D, keyboard_parts:D_SOD123_axial, B.Cu at (401.7, 223.0)
- added K_55: KEYSW, keyswitches:Kailh_socket_MX_led stab, F.Cu at (395.1, 239.0)
- added REF**: D_5W_P5.08mm_Vertical_AnodeUp, Diode_THT:D_5W_P5.08mm_Vertical_AnodeUp, F.Cu at (447.1, 168.3)
- added REF**: PinHeader_1x06_P2.54mm_Vertical, Connector_PinHeader_2.54mm:PinHeader_1x06_P2.54mm_Vertical, F.Cu at (248.4, 268.1)
- REF**: value PinHeader_1x12_P2.54mm_Vertical -> PinHeader_1x05_P2.54mm_Vertical; footprint Connector_PinHeader_2.54mm:PinHeader_1x12_P2.54mm_Vertical -> Connector_PinHeader_2.54mm:PinHeader_1x05_P2.54mm_Vertical
- moved REF** 17.8 mm to (300.1, 264.0)
Routing:
- net (no net): track 4735.3 -> 6307.3 mm, vias 8 -> 10
Other:
- board text added: "|<---Col 0-11--->|"
- board text added: "|<-Col 12-14,encoder->|"
- board text added: "|<-Row 0-5->|"
