File: 75% rev2/pcb/mcu daughterboard/mcu daughterboard.kicad_pcb (KiCad board)
At the start: 2 copper layers, 32.2 x 36.7 mm, 18 parts, among them U1 ATMEGA32U4, X1 XTAL_GND

Commit message: pcb file update
Parts:
- REF**: value MountingHole_2.2mm_M2_DIN965 -> .
Other:
- board text added: "GND"
- board text added: "Reset"
- board text added: "VCC"
- board text added: "encoder"
- board text added: "|<----Col 0-11---->|"
- board text added: "|<Col 12-15>|"
- board text added: "|<Row 0-6>|"
Changed lines of the file:
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@@
         (effects (font (size 1 1) (thickness 0.15)))
     )
-    (fp_text value "MountingHole_2.2mm_M2_DIN965" (at 0 2.9) (layer "Cmts.User") hide
+    (fp_text value "." (at 0 2.9) (layer "Cmts.User") hide
         (effects (font (size 1 1) (thickness 0.15)))
     )
@@
   (gr_line (start 155.638558 87.2137) (end 155.638558 117.9537)
     (stroke (width 0.1) (type default)) (layer "Edge.Cuts"))
-  (gr_arc (start 140.1325 143.4825) (mid 140.1325 143.4825) (end 140.1325 143.4825)
-    (stroke (width 0.2) (type solid)) (layer "Edge.Cuts"))
   (gr_line (start 152.638558 120.9537) (end 126.388558 120.9537)
     (stroke (width 0.1) (type default)) (layer "Edge.Cuts"))
@@
   (gr_arc (start 126.388558 120.9537) (mid 124.267265 120.075005) (end 123.388558 117.9537)
     (stroke (width 0.1) (type default)) (layer "Edge.Cuts"))
+  (gr_text "GND" (at 135.78 116.69) (layer "B.SilkS")
+    (effects (font (size 1 0.75) (thickness 0.125)) (justify left bottom mirror))
+  )
+  (gr_text "VCC" (at 143.03 116.94) (layer "B.SilkS")
+    (effects (font (size 1 0.75) (thickness 0.1875)) (justify left bottom mirror))
+  )
+  (gr_text "|<----Col 0-11---->|" (at 124.76 120.35 90) (layer "F.SilkS")
+    (effects (font (size 1 1.5) (thickness 0.1875)) (justify left bottom))
+  )
+  (gr_text "encoder" (at 133.83 90.79) (layer "F.SilkS")
+    (effects (font (size 0.5 0.5) (thickness 0.125)) (justify left bottom))
+  )
+  (gr_text "|<Row 0-6>|" (at 137.72 88.94) (layer "F.SilkS")
+    (effects (font (size 1 1.5) (thickness 0.125)) (justify left bottom))
+  )
+  (gr_text "Reset" (at 149.49 94.78) (layer "F.SilkS")
+    (effects (font (size 1 1.5) (thickness 0.125)) (justify left bottom))
+  )
+  (gr_text "|<Col 12-15>|" (at 124.298558 88.854804) (layer "F.SilkS")
+    (effects (font (size 1 0.75) (thickness 0.1875)) (justify left bottom))
+  )
+  (gr_text "encoder" (at 134.29 85.14) (layer "F.SilkS")
+    (effects (font (size 0.5 0.5) (thickness 0.125)) (justify left bottom))
+  )
   (segment (start 153.953558 102.092304) (end 153.953558 92.842304) (width 0.25) (layer "F.Cu") (net 0))
   (segment (start 153.953558 92.842304) (end 153.548558 92.437304) (width 0.25) (layer "F.Cu") (net 0))

Commit message: updates
Parts:
- moved * 0.72 mm to (135.8, 88.8)
Routing:
- net Net-(U1-Pad43): track 7.46 -> 10.3 mm
- net Net-(U1-Pad42): track 10.9 -> 10.1 mm
Other:
- board text added: "Befuddled"
- board text added: "D+"
- board text added: "D-"
