File: My75/My75 Rev2/pcb/main board/_autosave-keyboard.kicad_pcb (KiCad board)
At the start: 2 copper layers, 319.6 x 133.8 mm, 172 parts

Commit message: trashtruck added
Routing:
- net (no net): track 6307.3 -> 6264.1 mm

Commit message: pcb update final
Parts:
- added ?: , MountingHole:MountingHole_2.2mm_M2, F.Cu at (456.3, 273.9)
- added ?: , MountingHole:MountingHole_2.2mm_M2, F.Cu at (143.5, 274.0)
- added ?: , MountingHole:MountingHole_2.2mm_M2, F.Cu at (456.2, 147.1)
- added ?: , MountingHole:MountingHole_2.2mm_M2, F.Cu at (143.6, 146.9)
Routing:
- net (no net): track 6264.1 -> 6269.1 mm

Commit message: render/animation update
Routing:
- net (no net): track 6269.1 -> 6268.4 mm
