File: TrashTruck/V2/PCB/Switchplate/switchplate.kicad_pcb (KiCad board)
At the start: 2 copper layers, 346.9 x 89.8 mm, 0 parts

Commit message: zxc
Parts:
- added REF**: MountingHole_2.2mm_M2, MountingHole:MountingHole_2.2mm_M2, F.Cu at (121.8, 134.9)
- added REF**: MountingHole_2.2mm_M2, MountingHole:MountingHole_2.2mm_M2, F.Cu at (309.5, 59.1)
- added REF**: MountingHole_2.2mm_M2, MountingHole:MountingHole_2.2mm_M2, F.Cu at (-30.2, 134.5)
- added REF**: MountingHole_2.2mm_M2, MountingHole:MountingHole_2.2mm_M2, F.Cu at (309.1, 134.8)
- added REF**: MountingHole_2.2mm_M2, MountingHole:MountingHole_2.2mm_M2, F.Cu at (120.1, 60.7)
- added REF**: MountingHole_2.2mm_M2, MountingHole:MountingHole_2.2mm_M2, F.Cu at (-31.0, 59.0)
Other:
- board size 346.9 x 89.8 mm -> 346.9 x 95 mm
