File: My75/My75 Rev1 [Final]/PCB files/keyboard.kicad_pcb (KiCad board)
At the start: 2 copper layers, 324.3 x 134.3 mm, 168 parts, among them U1 Elite-C

Commit message: update
Routing:
- net (no net): track 6166.7 -> 6135.7 mm
- net /col16: track 112.8 -> 112.3 mm
Other:
- outline, holes or cut-outs redrawn
