File: TrashTruck/V2/PCB/TrashTruckV2/keyboard.kicad_pcb (KiCad board)
At the start: 2 copper layers, 350.9 x 93.7 mm, 114 parts

Commit message: trash update
Parts:
- removed D_0, D_1, D_10, D_11, D_12, D_13, D_14, D_15, D_16, D_17, D_18, D_19, D_2, D_20, D_21, D_22, D_23, D_24, D_25, D_26, D_27, D_28, D_29, D_3, D_30, D_31, D_32, D_33, D_34, D_35, D_36, D_37, D_38, D_39, D_4, D_40, D_41, D_42, D_43, D_44, D_45, D_46, D_47, D_48, D_49, D_5, D_50, D_51, D_52, D_53, D_54, D_55, D_56, D_6, D_7, D_8, D_9: D, Diode_SMD:D_SOD-123
- added REF**: RotaryEncoder_Alps_EC11E-Switch_Vertical_H20mm, Rotary_Encoder:RotaryEncoder_Alps_EC11E-Switch_Vertical_H20mm, F.Cu at (382.6, 168.2)
- added REF**: PinHeader_1x03_P2.54mm_Vertical, Connector_PinHeader_2.54mm:PinHeader_1x03_P2.54mm_Vertical, F.Cu at (387.9, 159.7)
- added REF**: D_A-405_P7.62mm_Horizontal, Diode_THT:D_A-405_P7.62mm_Horizontal, F.Cu at (165.8, 221.6)
- added REF**: D_A-405_P7.62mm_Horizontal, Diode_THT:D_A-405_P7.62mm_Horizontal, F.Cu at (366.0, 202.3)
- added REF**: D_A-405_P7.62mm_Horizontal, Diode_THT:D_A-405_P7.62mm_Horizontal, F.Cu at (244.6, 221.4)
- added REF**: D_A-405_P7.62mm_Horizontal, Diode_THT:D_A-405_P7.62mm_Horizontal, F.Cu at (142.1, 221.4)
- added REF**: D_A-405_P7.62mm_Horizontal, Diode_THT:D_A-405_P7.62mm_Horizontal, F.Cu at (142.1, 183.3)
- added REF**: PinHeader_1x16_P2.54mm_Vertical, Connector_PinHeader_2.54mm:PinHeader_1x16_P2.54mm_Vertical, F.Cu at (378.6, 188.6)
- added REF**: D_A-405_P7.62mm_Horizontal, Diode_THT:D_A-405_P7.62mm_Horizontal, F.Cu at (323.2, 221.5)
- added REF**: PinHeader_1x04_P2.54mm_Vertical, Connector_PinHeader_2.54mm:PinHeader_1x04_P2.54mm_Vertical, F.Cu at (395.5, 152.3)
- added REF**: D_A-405_P7.62mm_Horizontal, Diode_THT:D_A-405_P7.62mm_Horizontal, F.Cu at (346.9, 221.3)
- added REF**: D_A-405_P7.62mm_Horizontal, Diode_THT:D_A-405_P7.62mm_Horizontal, F.Cu at (146.9, 202.6)
- added REF**: D_A-405_P7.62mm_Horizontal, Diode_THT:D_A-405_P7.62mm_Horizontal, F.Cu at (361.3, 183.3)
- K_0, K_1, K_10, K_11, K_12, K_13, K_14, K_15, K_17, K_18, K_19, K_2, K_20, K_21, K_22, K_23, K_24, K_25, K_26, K_28, K_29, K_3, K_30, K_32, K_33, K_34, K_35, K_36, K_37, K_38, K_39, K_4, K_40, K_41, K_43, K_44, K_45, K_46, K_5, K_52, K_53, K_54, K_55, K_56, K_6, K_7, K_8, K_9: footprint MX_Alps_Hybrid:MX-1U-NoLED -> MX_Alps_Hybrid-master:hotswap with diode
- K_16, K_42, K_47, K_48, K_50, K_51: footprint MX_Alps_Hybrid:MX-1.25U-NoLED -> MX_Alps_Hybrid-master:MXOnly-1.25U-Hotswap
- K_27, K_31: footprint MX_Alps_Hybrid:MX-1.75U-NoLED -> MX_Alps_Hybrid-master:MXOnly-1.75U-Hotswap
- K_49: footprint MX_Alps_Hybrid:MX-7U-NoLED -> MX_Only:MXOnly-7U-Hotswap
- moved K_23 194.5 mm to (270.3, 179.6)
- moved K_28 194.5 mm to (417.9, 179.6)
- moved K_29 194.5 mm to (437.0, 179.6)
- moved K_40 194.5 mm to (317.9, 198.6)
- moved K_43 194.5 mm to (417.9, 198.6)
- moved K_44 194.5 mm to (437.0, 198.6)
- moved K_52 194.5 mm to (437.0, 217.7)
- moved K_55 194.5 mm to (389.3, 227.2)
- moved K_0 194.5 mm to (132.2, 160.5)
- moved K_1 194.5 mm to (151.2, 160.5)
- moved K_10 194.5 mm to (322.7, 160.5)
- moved K_11 194.5 mm to (341.7, 160.5)
- moved K_13 194.5 mm to (417.9, 160.5)
- moved K_14 194.5 mm to (437.0, 160.5)
- moved K_17 194.5 mm to (156.0, 179.6)
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Connections:
- K_0 pad 1: col0 -> (no net)
- K_0 pad 2: Net-(D_0-Pad2) -> (no net)
- K_1 pad 1: col1 -> (no net)
- K_1 pad 2: Net-(D_1-Pad2) -> (no net)
- K_10 pad 1: col10 -> (no net)
- K_10 pad 2: Net-(D_10-Pad2) -> (no net)
- K_11 pad 1: col11 -> (no net)
- K_11 pad 2: Net-(D_11-Pad2) -> (no net)
- K_12 pad 1: col12 -> (no net)
- K_12 pad 2: Net-(D_12-Pad2) -> (no net)
- K_13 pad 1: col15 -> (no net)
- K_13 pad 2: Net-(D_13-Pad2) -> (no net)
- K_14 pad 1: col16 -> (no net)
- K_14 pad 2: Net-(D_14-Pad2) -> (no net)
- K_15 pad 1: col17 -> (no net)
- K_15 pad 2: Net-(D_15-Pad2) -> (no net)
- K_16 pad 1: col0 -> (no net)
- K_16 pad 2: Net-(D_16-Pad2) -> (no net)
- K_17 pad 1: col1 -> (no net)
- K_17 pad 2: Net-(D_17-Pad2) -> (no net)
- K_18 pad 1: col2 -> (no net)
- K_18 pad 2: Net-(D_18-Pad2) -> (no net)
- K_19 pad 1: col3 -> (no net)
- K_19 pad 2: Net-(D_19-Pad2) -> (no net)
- K_2 pad 1: col2 -> (no net)
- K_2 pad 2: Net-(D_2-Pad2) -> (no net)
- K_20 pad 1: col4 -> (no net)
- K_20 pad 2: Net-(D_20-Pad2) -> (no net)
- K_21 pad 1: col5 -> (no net)
- K_21 pad 2: Net-(D_21-Pad2) -> (no net)
- K_22 pad 1: col6 -> (no net)
- K_22 pad 2: Net-(D_22-Pad2) -> (no net)
- K_23 pad 1: col7 -> (no net)
- K_23 pad 2: Net-(D_23-Pad2) -> (no net)
- K_24 pad 1: col8 -> (no net)
- K_24 pad 2: Net-(D_24-Pad2) -> (no net)
- K_25 pad 1: col9 -> (no net)
- K_25 pad 2: Net-(D_25-Pad2) -> (no net)
- K_26 pad 1: col10 -> (no net)
- K_26 pad 2: Net-(D_26-Pad2) -> (no net)
- K_27 pad 1: col12 -> (no net)
- K_27 pad 2: Net-(D_27-Pad2) -> (no net)
- K_28 pad 1: col15 -> (no net)
- K_28 pad 2: Net-(D_28-Pad2) -> (no net)
- K_29 pad 1: col16 -> (no net)
- K_29 pad 2: Net-(D_29-Pad2) -> (no net)
- K_3 pad 1: col3 -> (no net)
- K_3 pad 2: Net-(D_3-Pad2) -> (no net)
- K_30 pad 1: col17 -> (no net)
- K_30 pad 2: Net-(D_30-Pad2) -> (no net)
- K_31 pad 1: col0 -> (no net)
- K_31 pad 2: Net-(D_31-Pad2) -> (no net)
- K_32 pad 1: col2 -> (no net)
- K_32 pad 2: Net-(D_32-Pad2) -> (no net)
- K_33 pad 1: col3 -> (no net)
- K_33 pad 2: Net-(D_33-Pad2) -> (no net)
- K_34 pad 1: col4 -> (no net)
- K_34 pad 2: Net-(D_34-Pad2) -> (no net)
- K_35 pad 1: col5 -> (no net)
- K_35 pad 2: Net-(D_35-Pad2) -> (no net)
- K_36 pad 1: col6 -> (no net)
- K_36 pad 2: Net-(D_36-Pad2) -> (no net)
- K_37 pad 1: col7 -> (no net)
- K_37 pad 2: Net-(D_37-Pad2) -> (no net)
- K_38 pad 1: col8 -> (no net)
- K_38 pad 2: Net-(D_38-Pad2) -> (no net)
- K_39 pad 1: col9 -> (no net)
- K_39 pad 2: Net-(D_39-Pad2) -> (no net)
- K_4 pad 1: col4 -> (no net)
- K_4 pad 2: Net-(D_4-Pad2) -> (no net)
- K_40 pad 1: col10 -> (no net)
- K_40 pad 2: Net-(D_40-Pad2) -> (no net)
- K_41 pad 1: col11 -> (no net)
- K_41 pad 2: Net-(D_41-Pad2) -> (no net)
- K_42 pad 1: col12 -> (no net)
- K_42 pad 2: Net-(D_42-Pad2) -> (no net)
- K_43 pad 1: col15 -> (no net)
- K_43 pad 2: Net-(D_43-Pad2) -> (no net)
- K_44 pad 1: col16 -> (no net)
- K_44 pad 2: Net-(D_44-Pad2) -> (no net)
- K_45 pad 1: col17 -> (no net)
- K_45 pad 2: Net-(D_45-Pad2) -> (no net)
- K_46 pad 1: col14 -> (no net)
- K_46 pad 2: Net-(D_46-Pad2) -> (no net)
- K_47 pad 1: col0 -> (no net)
- K_47 pad 2: Net-(D_47-Pad2) -> (no net)
- K_48 pad 1: col1 -> (no net)
- K_48 pad 2: Net-(D_48-Pad2) -> (no net)
- K_49 pad 1: col6 -> (no net)
- K_49 pad 2: Net-(D_49-Pad2) -> (no net)
- K_5 pad 1: col5 -> (no net)
- K_5 pad 2: Net-(D_5-Pad2) -> (no net)
- K_50 pad 1: col10 -> (no net)
- K_50 pad 2: Net-(D_50-Pad2) -> (no net)
- K_51 pad 1: col11 -> (no net)
- K_51 pad 2: Net-(D_51-Pad2) -> (no net)
- K_52 pad 1: col16 -> (no net)
- K_52 pad 2: Net-(D_52-Pad2) -> (no net)
- K_53 pad 1: col17 -> (no net)
- K_53 pad 2: Net-(D_53-Pad2) -> (no net)
- K_54 pad 1: col13 -> (no net)
- K_54 pad 2: Net-(D_54-Pad2) -> (no net)
- K_55 pad 1: col14 -> (no net)
- K_55 pad 2: Net-(D_55-Pad2) -> (no net)
- K_56 pad 1: col15 -> (no net)
- K_56 pad 2: Net-(D_56-Pad2) -> (no net)
- K_6 pad 1: col6 -> (no net)
- K_6 pad 2: Net-(D_6-Pad2) -> (no net)
- K_7 pad 1: col7 -> (no net)
- K_7 pad 2: Net-(D_7-Pad2) -> (no net)
- K_8 pad 1: col8 -> (no net)
- K_8 pad 2: Net-(D_8-Pad2) -> (no net)
- K_9 pad 1: col9 -> (no net)
- K_9 pad 2: Net-(D_9-Pad2) -> (no net)
Routing:
- net (no net): track 0.00 -> 3993.1 mm, vias 0 -> 2
- added copper zone on B.Cu, net (none)
- added copper zone on F.Cu, net (none)
Other:
- outline, holes or cut-outs redrawn

Commit message: trash
Routing:
- net (no net): track 3993.1 -> 4534.2 mm, vias 2 -> 4

Commit message: pcb update
Parts:
- added REF**: D_A-405_P7.62mm_Horizontal, Diode_THT:D_A-405_P7.62mm_Horizontal, F.Cu at (399.1, 180.8)
Routing:
- net (no net): track 4534.2 -> 6437.8 mm, vias 4 -> 17

Commit message: documentation
Routing:
- net (no net): track 6437.8 -> 6439.2 mm, vias 17 -> 23

Commit message: zxc
Parts:
- added REF**: MountingHole_2.2mm_M2, MountingHole:MountingHole_2.2mm_M2, F.Cu at (464.4, 151.7)
- added REF**: MountingHole_2.2mm_M2, MountingHole:MountingHole_2.2mm_M2, F.Cu at (275.1, 153.3)
- added REF**: MountingHole_2.2mm_M2, MountingHole:MountingHole_2.2mm_M2, F.Cu at (123.9, 151.6)
- added REF**: MountingHole_2.2mm_M2, MountingHole:MountingHole_2.2mm_M2, F.Cu at (464.1, 227.5)
- added REF**: MountingHole_2.2mm_M2, MountingHole:MountingHole_2.2mm_M2, F.Cu at (124.8, 227.1)
- added REF**: MountingHole_2.2mm_M2, MountingHole:MountingHole_2.2mm_M2, F.Cu at (276.7, 227.5)
Routing:
- net (no net): track 6439.2 -> 6437.7 mm
