File: Alicida/top pl/top pl.kicad_pcb (KiCad board)
At the start: 2 copper layers, 380.4 x 120.4 mm, 62 parts

Commit message: fghyuj
Routing:
- added copper zone on B.Cu, net (none)
- added copper zone on F.Cu, net (none)
