File: Keyjoy/pcb/top plate/top plate.kicad_pcb (KiCad board)
At the start: 2 copper layers, 333.9 x 125 mm, 128 parts

Commit message: sefg
Parts:
- moved K_SPACE2 13.3 mm to (366.8, 245.6)
Changed lines of the file:
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@@
       (stroke (width 0.1) (type solid)) (layer "Dwgs.User"))
     (fp_line (start -15.311 -5.52) (end -15.311 6.78)
-      (stroke (width 0.1) (type solid)) (layer "Eco1.User"))
+      (stroke (width 0.1) (type solid)) (layer "Edge.Cuts"))
     (fp_line (start -15.311 6.78) (end -8.561 6.78)
-      (stroke (width 0.1) (type solid)) (layer "Eco1.User"))
+      (stroke (width 0.1) (type solid)) (layer "Edge.Cuts"))
     (fp_line (start -8.561 -5.52) (end -15.311 -5.52)
-      (stroke (width 0.1) (type solid)) (layer "Eco1.User"))
+      (stroke (width 0.1) (type solid)) (layer "Edge.Cuts"))
     (fp_line (start -8.561 6.78) (end -8.561 -5.52)
-      (stroke (width 0.1) (type solid)) (layer "Eco1.User"))
+      (stroke (width 0.1) (type solid)) (layer "Edge.Cuts"))
     (fp_line (start 8.565 -5.52) (end 8.565 6.78)
-      (stroke (width 0.1) (type solid)) (layer "Eco1.User"))
+      (stroke (width 0.1) (type solid)) (layer "Edge.Cuts"))
     (fp_line (start 8.565 6.78) (end 15.315 6.78)
-      (stroke (width 0.1) (type solid)) (layer "Eco1.User"))
+      (stroke (width 0.1) (type solid)) (layer "Edge.Cuts"))
     (fp_line (start 15.315 -5.52) (end 8.565 -5.52)
-      (stroke (width 0.1) (type solid)) (layer "Eco1.User"))
+      (stroke (width 0.1) (type solid)) (layer "Edge.Cuts"))
     (fp_line (start 15.315 6.78) (end 15.315 -5.52)
-      (stroke (width 0.1) (type solid)) (layer "Eco1.User"))
+      (stroke (width 0.1) (type solid)) (layer "Edge.Cuts"))
     (fp_rect (start -15.3 -5.52) (end -8.58 6.76)
       (stroke (width 0.05) (type default)) (fill none) (layer "Edge.Cuts"))
@@
         (effects (font (size 1 1) (thickness 0.15)))
     )
-    (fp_text user "${REFERENCE}" (at 0 2.455 unlocked) (layer "F.Fab")
+    (fp_text user "${REFERENCE}" (at 0 2.455 unlocked) (layer "F.Fab") hide
         (effects (font (size 1 1) (thickness 0.15)))
     )
@@
   )
   (footprint "Switch_Keyboard_Hotswap_Kailh:SW_Kailh_MX_top plate" (layer "F.Cu")
-    (at 377.573021 253.329898)
+    (at 366.804312 245.590264)
     (descr "Kailh keyswitch Hotswap Socket")
     (tags "Kailh Keyboard Keyswitch Switch Hotswap Socket Relief Cutout")
@@
   (gr_arc (start 477.950644 151.645592) (mid 481.600798 153.073089) (end 483.089978 156.698516)
     (stroke (width 0.1) (type default)) (layer "Edge.Cuts"))
-  (gr_arc (start 149.25009 154.797334) (mid 149.25009 154.797334) (end 149.25009 154.797334)
-    (stroke (width 0.2) (type solid)) (layer "Edge.Cuts"))
   (gr_line (start 180.307428 151.698516) (end 451.89535 151.710799)
     (stroke (width 0.1) (type default)) (layer "Edge.Cuts"))
@@
   (gr_line (start 180.307428 146.562095) (end 180.307428 151.698516)
     (stroke (width 0.1) (type default)) (layer "Edge.Cuts"))
-  (zone (net 0) (net_name "") (layer "F.Cu") (hatch edge 0.508)
-    (connect_pads yes (clearance 0.25))
-    (min_thickness 0.254) (filled_areas_thickness no)
-    (fill yes (thermal_gap 0.508) (thermal_bridge_width 0.508))
+  (zone (net 0) (net_name "") (layer "F.Cu") (hatch edge 0.5)
+    (connect_pads (clearance 0.508))
+    (min_thickness 0.25) (filled_areas_thickness no)
+    (fill (thermal_gap 0.5) (thermal_bridge_width 0.5) (island_removal_mode 1) (island_area_min 10))
     (polygon
       (pts
-        (xy 138.840018 138.573588)
-        (xy 140.726894 277.105969)
-        (xy 487.055278 278.339294)
-        (xy 485.168402 139.806913)
+        (xy 136.796302 124.771246)
+        (xy 492.177244 127.716391)
+        (xy 491.195529 281.354838)
+        (xy 135.814586 281.354838)
       )
     )
   )
-  (zone (net 0) (net_name "") (layer "B.Cu") (hatch edge 0.508)
-    (connect_pads yes (clearance 0.25))
-    (min_thickness 0.254) (filled_areas_thickness no)
-    (fill yes (thermal_gap 0.508) (thermal_bridge_width 0.508))
+  (zone (net 0) (net_name "") (layer "B.Cu") (hatch edge 0.5)
+    (priority 1)
+    (connect_pads (clearance 0.508))
+    (min_thickness 0.25) (filled_areas_thickness no)
+    (fill (thermal_gap 0.5) (thermal_bridge_width 0.5) (island_removal_mode 1) (island_area_min 10))
     (polygon
       (pts
-        (xy 140.844291 139.535061)
-        (xy 141.555887 278.788875)
-        (xy 486.351096 278.884543)
-        (xy 485.6395 139.630729)
+        (xy 136.796302 124.771246)
+        (xy 492.177244 127.716391)
+        (xy 491.195529 281.354838)
+        (xy 135.814586 281.354838)
       )
     )

Commit message: fab update
Parts:
- removed the REF** at (418.6, 207.6)
- removed the REF** at (175.7, 225.8)
- removed the REF** at (421.0, 169.3)
- removed REFr: top plate stab, Switch_Keyboard_Hotswap_Kailh:top plate stab
- added REF**: top plate stab, Mounting_Keyboard_Stabilizer:top plate stab, F.Cu at (412.3, 211.6)
- added REF**: nothing, personal:nothing, B.Cu at (177.0, 192.3)
- added REF**: nothing, personal:nothing, B.Cu at (291.1, 230.7)
- added REF**: nothing, personal:nothing, B.Cu at (181.7, 211.7)
- added REF**: nothing, personal:nothing, B.Cu at (424.6, 192.4)
- added REF**: nothing, personal:nothing, B.Cu at (195.9, 230.6)
- added REF**: nothing, personal:nothing, B.Cu at (172.1, 230.7)
- added REF**: top plate stab, Mounting_Keyboard_Stabilizer:top plate stab, F.Cu at (419.4, 154.4)
- added REF**: top plate stab, Mounting_Keyboard_Stabilizer:top plate stab, F.Cu at (174.1, 211.6)
- added REF**: top plate stab, Mounting_Keyboard_Stabilizer:top plate stab, F.Cu at (417.0, 192.6)
- added REF**: nothing, personal:nothing, B.Cu at (174.7, 173.4)
- added REF**: nothing, personal:nothing, B.Cu at (431.8, 173.4)
- added REF**: nothing, personal:nothing, B.Cu at (219.7, 230.8)
- added REF**: nothing, personal:nothing, B.Cu at (427.0, 154.4)
- added REF**: nothing, personal:nothing, B.Cu at (419.6, 211.7)
- moved K_SPACE2 15.6 mm to (362.2, 230.7)
- moved D_0 14.9 mm to (362.7, 155.0)
- moved D_1 14.9 mm to (191.3, 155.0)
- moved D_2 14.9 mm to (210.3, 155.0)
- moved D_4 14.9 mm to (248.4, 155.0)
- moved D_5 14.9 mm to (267.5, 155.0)
- moved D_6 14.9 mm to (286.5, 155.0)
- moved D_8 14.9 mm to (324.6, 155.0)
- moved D_9 14.9 mm to (343.7, 155.0)
- moved D_ALT 14.9 mm to (224.6, 231.2)
- moved D_B 14.9 mm to (291.3, 212.1)
- moved D_BACKSPACE 14.9 mm to (438.9, 155.0)
- moved D_BSLSH 14.9 mm to (438.9, 174.0)
- moved D_CAPS 14.9 mm to (186.5, 193.1)
- moved D_CBRAC 14.9 mm to (391.3, 174.0)
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Other:
- board size 333.9 x 125 mm -> 333.9 x 122.4 mm

Commit message: 3d update
Other:
- board text added: "Keyjoy - By: Skycode22"
