File: Store Boards/Keyjoy/pcb/keyjoy/keyjoy.kicad_pcb (KiCad board)
At the start: 2 copper layers, 333.9 x 114.7 mm, 143 parts

Commit message: pcb update
Routing:
- net (no net): track 7986.2 -> 8039.0 mm, vias 21 -> 25
