File: Store Boards/Keyjoy/pcb/top plate/top plate.kicad_pcb (KiCad board)
At the start: 2 copper layers, 333.9 x 122.4 mm, 139 parts

Commit message: pcb update
Parts:
- added ?: , , F.Cu at (471.9, 218.2)
- added ?: , , F.Cu at (477.4, 140.4)
- added ?: , , F.Cu at (233.6, 183.1)
- added REF**: MountingHole_2.2mm_M2, MountingHole:MountingHole_2.2mm_M2, F.Cu at (433.1, 241.6)
- added REF**: MountingHole_2.2mm_M2, MountingHole:MountingHole_2.2mm_M2, F.Cu at (309.4, 141.0)
- added REF**: MountingHole_2.2mm_M2, MountingHole:MountingHole_2.2mm_M2, F.Cu at (471.9, 218.2)
- added REF**: MountingHole_2.2mm_M2, MountingHole:MountingHole_2.2mm_M2, F.Cu at (477.4, 140.4)
- added REF**: MountingHole_2.2mm_M2, MountingHole:MountingHole_2.2mm_M2, F.Cu at (151.5, 140.5)
- added REF**: MountingHole_2.2mm_M2, MountingHole:MountingHole_2.2mm_M2, F.Cu at (308.3, 243.3)
- added REF**: MountingHole_2.2mm_M2, MountingHole:MountingHole_2.2mm_M2, F.Cu at (151.7, 248.1)
- added REF**: MountingHole_2.2mm_M2, MountingHole:MountingHole_2.2mm_M2, F.Cu at (358.3, 183.2)
- added REF**: MountingHole_2.2mm_M2, MountingHole:MountingHole_2.2mm_M2, F.Cu at (233.6, 183.1)
