File: Store Boards/Track75/pcb/keyboard.kicad_pcb (KiCad board)
At the start: 2 copper layers, 349.2 x 105.6 mm, 152 parts, among them IC1 AP7335-WG-7, J1 Conn_01x06_Female, U1 XC6206P332MR, U2 PMW3360DM-T2QU, U4 TXS0104EDR

Commit message: update
Parts:
- removed D_CTRL1, D_DOWN, D_LEFT, D_RIGHT, D_UP: D, personal:nothing
- removed K_CTRL1, K_LEFT, K_UP: KEYSW, personal:1u mx hotswap with diode
- added REF**: MountingHole_3.2mm_M3, MountingHole:MountingHole_3.2mm_M3, F.Cu at (35.2, 213.6)
- added REF**: MountingHole_3.2mm_M3, MountingHole:MountingHole_3.2mm_M3, F.Cu at (390.0, 213.7)
- added REF**: MountingHole_2.2mm_M2, MountingHole:MountingHole_2.2mm_M2, F.Cu at (124.7, 134.5)
- added REF**: MountingHole_2.2mm_M2, MountingHole:MountingHole_2.2mm_M2, F.Cu at (222.4, 134.6)
- added REF**: MountingHole_3.2mm_M3, MountingHole:MountingHole_3.2mm_M3, F.Cu at (390.1, 114.9)
- added REF**: MountingHole_2.2mm_M2, MountingHole:MountingHole_2.2mm_M2, F.Cu at (45.5, 134.5)
- added REF**: MountingHole_3.2mm_M3, MountingHole:MountingHole_3.2mm_M3, F.Cu at (34.8, 115.6)
- added REF**: PinHeader_1x03_P2.54mm_Vertical, Connector_PinHeader_2.54mm:PinHeader_1x03_P2.54mm_Vertical, F.Cu at (385.3, 190.2)
- added REF**: RPi_Pico_SMD_TH, MCU_RaspberryPi_and_Boards:RPi_Pico_SMD_TH, B.Cu at (353.6, 124.8)
- added REF**: MountingHole_2.2mm_M2, MountingHole:MountingHole_2.2mm_M2, F.Cu at (387.6, 133.0)
- added REF**: MountingHole_2.2mm_M2, MountingHole:MountingHole_2.2mm_M2, F.Cu at (301.5, 134.3)
- added REF**: XDCR_COM-09032, PS4_joystick_footprint-main:PS4_joystick, F.Cu at (298.8, 207.0)
- added REF**: MountingHole_2.2mm_M2, MountingHole:MountingHole_2.2mm_M2, F.Cu at (348.8, 189.6)
- added REF**: MountingHole_2.2mm_M2, MountingHole:MountingHole_2.2mm_M2, F.Cu at (76.2, 190.0)
- added REF**: MountingHole_2.2mm_M2, MountingHole:MountingHole_2.2mm_M2, F.Cu at (199.9, 191.6)
- moved C1 46.5 mm to (370.5, 174.5)
- moved R1 46.5 mm to (370.5, 160.5)
- moved R2 46.5 mm to (364.0, 145.7)
- moved R3 46.5 mm to (366.6, 145.7)
- moved R4 46.5 mm to (362.4, 170.8)
- moved C2 46.5 mm to (370.5, 164.8)
- moved C5 46.5 mm to (370.4, 145.8)
- moved IC1 46.5 mm to (370.4, 151.8)
- moved U4 46.5 mm to (347.8, 157.0)
- moved C3 46.5 mm to (349.4, 166.3)
- moved C4 46.5 mm to (370.5, 156.4)
- moved J1 46.5 mm to (377.3, 153.9)
- moved U1 46.5 mm to (375.1, 169.6)
- moved U2 46.5 mm to (355.1, 168.0)
- moved D_0 42.0 mm to (245.1, 125.4)
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Routing:
- net (no net): track 485.4 -> 6754.6 mm, vias 8 -> 20
- added copper zone on F.Cu, net GND
- removed copper zone on F.Cu, net (none)
Other:
- board size 349.2 x 105.6 mm -> 364.9 x 108.3 mm

Commit message: kicad update
Connections:
- REF** pad 38: (no net) -> GND
Routing:
- net (no net): track 6754.6 -> 7124.2 mm, vias 20 -> 29
- net GND: track 29.8 -> 63.0 mm
