File: keyboards in progress/60new/Kicad/keyboard.kicad_pcb (KiCad board)
At the start: 2 copper layers, 362.4 x 105.2 mm, 141 parts, among them SW1 SW_PUSH, U1 ATMEGA32U4, X1 XTAL_GND

Commit message: new keyboard
Parts:
- added C1: 2.2uF, Capacitor_SMD:C_1206_3216Metric_Pad1.42x1.75mm_HandSolder, B.Cu at (449.5, 208.1)
- added C2: 10uF, Capacitor_SMD:C_1206_3216Metric_Pad1.42x1.75mm_HandSolder, B.Cu at (449.5, 198.4)
- added C3: 4.7uF, Capacitor_SMD:C_1206_3216Metric_Pad1.42x1.75mm_HandSolder, B.Cu at (428.5, 199.9)
- added C4: 1uF, Capacitor_SMD:C_1206_3216Metric_Pad1.42x1.75mm_HandSolder, B.Cu at (449.5, 190.0)
- added C5: 1uF, Capacitor_SMD:C_1206_3216Metric_Pad1.42x1.75mm_HandSolder, B.Cu at (449.5, 179.4)
- added IC1: AP7335-WG-7, local:AP7331, B.Cu at (449.5, 185.4)
- added J1: Conn_01x06_Female, Connector_PinHeader_2.54mm:PinHeader_1x06_P2.54mm_Vertical, F.Cu at (456.3, 187.5)
- added R1: 10k, Resistor_SMD:R_1206_3216Metric_Pad1.42x1.75mm_HandSolder, B.Cu at (449.5, 194.1)
- added R2: 10k, Resistor_SMD:R_1206_3216Metric_Pad1.42x1.75mm_HandSolder, B.Cu at (443.0, 179.3)
- added R3: 15k, Resistor_SMD:R_1206_3216Metric_Pad1.42x1.75mm_HandSolder, B.Cu at (445.7, 179.3)
- added R4: 39, Resistor_SMD:R_1206_3216Metric_Pad1.42x1.75mm_HandSolder, B.Cu at (441.4, 204.4)
- added REF**: MountingHole_2.2mm_M2, MountingHole:MountingHole_2.2mm_M2, F.Cu at (299.9, 166.0)
- added REF**: MountingHole_2.2mm_M2, MountingHole:MountingHole_2.2mm_M2, F.Cu at (474.3, 145.6)
- added REF**: RotaryEncoder_Alps_EC11E-Switch_Vertical_H20mm, Rotary_Encoder:RotaryEncoder_Alps_EC11E-Switch_Vertical_H20mm, F.Cu at (431.4, 154.1)
- added REF**: MountingHole_2.2mm_M2, MountingHole:MountingHole_2.2mm_M2, F.Cu at (119.6, 145.8)
- added REF**: MountingHole_2.2mm_M2, MountingHole:MountingHole_2.2mm_M2, F.Cu at (293.1, 243.2)
- added REF**: MountingHole_2.2mm_M2, MountingHole:MountingHole_2.2mm_M2, F.Cu at (232.5, 185.2)
- added REF**: MountingHole_2.2mm_M2, MountingHole:MountingHole_2.2mm_M2, F.Cu at (119.3, 243.6)
- added REF**: MountingHole_2.2mm_M2, MountingHole:MountingHole_2.2mm_M2, F.Cu at (474.1, 243.3)
- added REF**: MountingHole_2.2mm_M2, MountingHole:MountingHole_2.2mm_M2, F.Cu at (365.6, 185.1)
- added U1: XC6206P332MR, Package_TO_SOT_SMD:TSOT-23_HandSoldering, B.Cu at (454.2, 203.2)
- added U2: PMW3360DM-T2QU, local:DIP-16_W10.16mm, B.Cu at (434.1, 201.6)
- added U4: TXS0104EDR, local:SOIC127P600X175-14N, B.Cu at (426.8, 190.6)
- USB1: footprint keyboard_parts:Molex-0548190589-Assembly -> Connector_USB:USB_C_Receptacle_Palconn_UTC16-G
- moved C1 29.6 mm to (454.8, 176.5)
- moved C2 29.6 mm to (464.8, 176.5)
- moved C3 29.6 mm to (454.8, 161.5)
- moved R1 29.6 mm to (463.8, 151.5)
- moved R2 29.6 mm to (474.8, 164.5)
- moved R3 29.6 mm to (454.8, 164.5)
- moved R4 29.6 mm to (454.8, 168.5)
- moved SW1 29.6 mm to (463.8, 146.5)
- moved U1 29.6 mm to (463.8, 161.5)
- moved X1 29.6 mm to (459.8, 176.5)
- moved C7 25.7 mm to (472.4, 173.4), turned to 90 degrees
- moved C6 20.5 mm to (472.4, 178.4), turned to 90 degrees
- moved C5 16.7 mm to (472.4, 183.4), turned to 90 degrees
- moved C4 15.4 mm to (472.4, 188.4), turned to 90 degrees
- moved USB1 2.61 mm to (299.5, 146.4), turned to 0 degrees
Routing:
- net (no net): track 0.00 -> 609.2 mm, vias 0 -> 10
- net GND: track 0.00 -> 29.8 mm, vias 0 -> 6
Other:
- outline, holes or cut-outs redrawn
- board text added: "+5V"
- board text added: "10k"
- board text added: "10u"
- board text added: "15k"
- board text added: "1u"
- board text added: "2.2u"
- board text added: "2V"
- board text added: "3.3V"
- board text added: "39"
- board text added: "4.7u"
- board text added: "5V"
- board text added: "ADJ"
- board text added: "EN"
- board text added: "GND"
- board text added: "MISO"
- board text added: "MOSI"
- board text added: "SCK"
- board text added: "SS"
- board text added: "Skycode22"
- board text removed: "PCB Builder by MisterKeebs - mrkeebs.com"

Commit message: update
Parts:
- removed the C1 at (454.8, 176.5)
- removed the C2 at (464.8, 176.5)
- removed the C3 at (454.8, 161.5)
- removed the C4 at (472.4, 188.4)
- removed the C5 at (472.4, 183.4)
- removed C6, C7: 22pF, Capacitor_SMD:C_0805_2012Metric_Pad1.15x1.40mm_HandSolder
- removed the R1 at (463.8, 151.5)
- removed the R2 at (474.8, 164.5)
- removed the R3 at (454.8, 164.5)
- removed the R4 at (454.8, 168.5)
- removed SW1: SW_PUSH, Button_Switch_SMD:SW_SPST_TL3342
- removed the U1 at (463.8, 161.5)
- removed USB1: Molex-0548190589, Connector_USB:USB_C_Receptacle_Palconn_UTC16-G
- removed X1: XTAL_GND, Crystal:Crystal_SMD_5032-4Pin_5.0x3.2mm
- K_0, K_1, K_2, K_3, K_4, K_5, K_6, K_7, K_8, K_9, K_A, K_B, K_C, K_CBRAC, K_COMMA, K_D, K_DOT, K_E, K_EQUAL, K_F, K_G, K_H, K_I, K_J, K_K, K_L, K_M, K_MINUS, K_N, K_O, K_OBRAC, K_P, K_Q, K_QUOTE, K_R, K_S, K_SEMIC, K_SLASH, K_SPACE, K_SPACE1, K_T, K_U, K_V, K_W, K_X, K_Y, K_Z, K_`: footprint MX_Alps_Hybrid:MX-1U-NoLED -> personal:1u mx hotswap with diode

Commit message: update
Parts:
- added ATMEGA32U4-AU: MCU**, hotswapmx:ATMEGA32U4-AU, F.Cu at (467.8, 182.5)
- added C1: 22pF, Capacitor_SMD:C_0805_2012Metric_Pad1.15x1.40mm_HandSolder, F.Cu at (474.8, 198.0)
- added C2: 22pF, Capacitor_SMD:C_0805_2012Metric_Pad1.15x1.40mm_HandSolder, F.Cu at (474.7, 193.4)
- added C3: 22pF, Capacitor_SMD:C_0805_2012Metric_Pad1.15x1.40mm_HandSolder, B.Cu at (454.6, 175.1)
- added C4: 22pF, Capacitor_SMD:C_0805_2012Metric_Pad1.15x1.40mm_HandSolder, B.Cu at (467.9, 179.6)
- added C5: 22pF, Capacitor_SMD:C_0805_2012Metric_Pad1.15x1.40mm_HandSolder, B.Cu at (469.5, 183.5)
- added C6: 22pF, Capacitor_SMD:C_0805_2012Metric_Pad1.15x1.40mm_HandSolder, B.Cu at (466.2, 182.0)
- added C7: 22pF, Capacitor_SMD:C_0805_2012Metric_Pad1.15x1.40mm_HandSolder, B.Cu at (466.3, 184.8)
- added R2: 10k, Resistor_SMD:R_0805_2012Metric_Pad1.15x1.40mm_HandSolder, B.Cu at (473.7, 175.9)
- added R3: 22, Resistor_SMD:R_0805_2012Metric_Pad1.15x1.40mm_HandSolder, B.Cu at (454.6, 178.1)
- added R4: 22, Resistor_SMD:R_0805_2012Metric_Pad1.15x1.40mm_HandSolder, B.Cu at (454.6, 182.1)
- added REF**: Stabilizer_MX_2u, hotswapmx:Stabilizer_MX_2u, F.Cu at (380.0, 213.8)
- added REF**: PinHeader_1x04_P2.54mm_Vertical, Connector_PinHeader_2.54mm:PinHeader_1x04_P2.54mm_Vertical, F.Cu at (453.6, 158.2)
- added REF**: Stabilizer_MX_2u, hotswapmx:Stabilizer_MX_2u, F.Cu at (141.9, 213.7)
- added REF**: Stabilizer_MX_2u, hotswapmx:Stabilizer_MX_2u, F.Cu at (387.2, 156.6)
- added REF**: Stabilizer_MX_2u, hotswapmx:Stabilizer_MX_2u, F.Cu at (384.8, 194.7)
- added X1: XTAL_GND, Crystal:Crystal_SMD_5032-4Pin_5.0x3.2mm, F.Cu at (469.7, 195.9)
- D_0, D_1, D_2, D_3, D_4, D_5, D_6, D_7, D_8, D_9, D_A, D_ALT, D_ALT1, D_B, D_BACKSPACE, D_BSLSH, D_C, D_CAPS, D_CBRAC, D_COMMA, D_CTRL, D_CTRL1, D_D, D_DOT, D_E, D_ENTER, D_EQUAL, D_F, D_G, D_H, D_I, D_J, D_K, D_L, D_M, D_MENU, D_MINUS, D_N, D_O, D_OBRAC, D_P, D_Q, D_QUOTE, D_R, D_S, D_SEMIC, D_SHIFT, D_SHIFT1, D_SLASH, D_SPACE, D_SPACE1, D_SPACE2, D_T, D_TAB, D_U, D_V, D_W, D_WIN, D_WIN1, D_X, D_Y, D_Z, D_`: footprint keyboard_parts:D_SOD123_axial -> personal:nothing
- K_ALT, K_ALT1, K_CTRL, K_CTRL1, K_MENU, K_WIN, K_WIN1: footprint MX_Alps_Hybrid:MX-1.25U-NoLED -> personal:1u mx hotswap with diode
- K_BACKSPACE: footprint MX_Alps_Hybrid:MX-2U-NoLED -> personal:1u mx hotswap with diode
- K_BSLSH, K_TAB: footprint MX_Alps_Hybrid:MX-1.5U-NoLED -> personal:1u mx hotswap with diode
- K_CAPS: footprint MX_Alps_Hybrid:MX-1.75U-NoLED -> personal:1u mx hotswap with diode
- K_ENTER, K_SHIFT: footprint MX_Alps_Hybrid:MX-2.25U-NoLED -> personal:1u mx hotswap with diode
- K_SHIFT1: footprint MX_Alps_Hybrid:MX-2.75U-NoLED -> personal:1u mx hotswap with diode
Connections:
- K_0 pad 1: /col10 -> (no net)
- K_0 pad 2: Net-(D_0-Pad2) -> (no net)
- K_1 pad 1: /col1 -> (no net)
- K_1 pad 2: Net-(D_1-Pad2) -> (no net)
- K_2 pad 1: /col2 -> (no net)
- K_2 pad 2: Net-(D_2-Pad2) -> (no net)
- K_3 pad 1: /col3 -> (no net)
- K_3 pad 2: Net-(D_3-Pad2) -> (no net)
- K_4 pad 1: /col4 -> (no net)
- K_4 pad 2: Net-(D_4-Pad2) -> (no net)
- K_5 pad 1: /col5 -> (no net)
- K_5 pad 2: Net-(D_5-Pad2) -> (no net)
- K_6 pad 1: /col6 -> (no net)
- K_6 pad 2: Net-(D_6-Pad2) -> (no net)
- K_7 pad 1: /col7 -> (no net)
- K_7 pad 2: Net-(D_7-Pad2) -> (no net)
- K_8 pad 1: /col8 -> (no net)
- K_8 pad 2: Net-(D_8-Pad2) -> (no net)
- K_9 pad 1: /col9 -> (no net)
- K_9 pad 2: Net-(D_9-Pad2) -> (no net)
- K_A pad 1: /col2 -> (no net)
- K_A pad 2: Net-(D_A-Pad2) -> (no net)
- K_ALT pad 1: /col3 -> (no net)
- K_ALT pad 2: Net-(D_ALT-Pad2) -> (no net)
- K_ALT1 pad 1: /col10 -> (no net)
- K_ALT1 pad 2: Net-(D_ALT1-Pad2) -> (no net)
- K_B pad 1: /col6 -> (no net)
- K_B pad 2: Net-(D_B-Pad2) -> (no net)
- K_BACKSPACE pad 1: /col14 -> (no net)
- K_BACKSPACE pad 2: Net-(D_BACKSPACE-Pad2) -> (no net)
- K_BSLSH pad 1: /col14 -> (no net)
- K_BSLSH pad 2: Net-(D_BSLSH-Pad2) -> (no net)
- K_C pad 1: /col4 -> (no net)
- K_C pad 2: Net-(D_C-Pad2) -> (no net)
- K_CAPS pad 1: /col0 -> (no net)
- K_CAPS pad 2: Net-(D_CAPS-Pad2) -> (no net)
- K_CBRAC pad 1: /col12 -> (no net)
- K_CBRAC pad 2: Net-(D_CBRAC-Pad2) -> (no net)
- K_COMMA pad 1: /col9 -> (no net)
- K_COMMA pad 2: Net-(D_COMMA-Pad2) -> (no net)
- K_CTRL pad 1: /col0 -> (no net)
- K_CTRL pad 2: Net-(D_CTRL-Pad2) -> (no net)
- K_CTRL1 pad 1: /col13 -> (no net)
- K_CTRL1 pad 2: Net-(D_CTRL1-Pad2) -> (no net)
- K_D pad 1: /col4 -> (no net)
- K_D pad 2: Net-(D_D-Pad2) -> (no net)
- K_DOT pad 1: /col10 -> (no net)
- K_DOT pad 2: Net-(D_DOT-Pad2) -> (no net)
- K_E pad 1: /col4 -> (no net)
- K_E pad 2: Net-(D_E-Pad2) -> (no net)
- K_ENTER pad 1: /col13 -> (no net)
- K_ENTER pad 2: Net-(D_ENTER-Pad2) -> (no net)
- K_EQUAL pad 1: /col12 -> (no net)
- K_EQUAL pad 2: Net-(D_EQUAL-Pad2) -> (no net)
- K_F pad 1: /col5 -> (no net)
- K_F pad 2: Net-(D_F-Pad2) -> (no net)
- K_G pad 1: /col6 -> (no net)
- K_G pad 2: Net-(D_G-Pad2) -> (no net)
- K_H pad 1: /col7 -> (no net)
- K_H pad 2: Net-(D_H-Pad2) -> (no net)
- K_I pad 1: /col9 -> (no net)
- K_I pad 2: Net-(D_I-Pad2) -> (no net)
- K_J pad 1: /col8 -> (no net)
- K_J pad 2: Net-(D_J-Pad2) -> (no net)
- K_K pad 1: /col9 -> (no net)
- K_K pad 2: Net-(D_K-Pad2) -> (no net)
- K_L pad 1: /col10 -> (no net)
- K_L pad 2: Net-(D_L-Pad2) -> (no net)
- K_M pad 1: /col8 -> (no net)
- K_M pad 2: Net-(D_M-Pad2) -> (no net)
- K_MENU pad 1: /col12 -> (no net)
- K_MENU pad 2: Net-(D_MENU-Pad2) -> (no net)
- K_MINUS pad 1: /col11 -> (no net)
- K_MINUS pad 2: Net-(D_MINUS-Pad2) -> (no net)
- K_N pad 1: /col7 -> (no net)
- K_N pad 2: Net-(D_N-Pad2) -> (no net)
- K_O pad 1: /col10 -> (no net)
- K_O pad 2: Net-(D_O-Pad2) -> (no net)
- K_OBRAC pad 1: /col13 -> (no net)
- K_OBRAC pad 2: Net-(D_OBRAC-Pad2) -> (no net)
- K_P pad 1: /col11 -> (no net)
- K_P pad 2: Net-(D_P-Pad2) -> (no net)
- K_Q pad 1: /col2 -> (no net)
- K_Q pad 2: Net-(D_Q-Pad2) -> (no net)
- K_QUOTE pad 1: /col12 -> (no net)
- K_QUOTE pad 2: Net-(D_QUOTE-Pad2) -> (no net)
- K_R pad 1: /col5 -> (no net)
- K_R pad 2: Net-(D_R-Pad2) -> (no net)
- K_S pad 1: /col3 -> (no net)
- K_S pad 2: Net-(D_S-Pad2) -> (no net)
- K_SEMIC pad 1: /col11 -> (no net)
- K_SEMIC pad 2: Net-(D_SEMIC-Pad2) -> (no net)
- K_SHIFT pad 1: /col1 -> (no net)
- K_SHIFT pad 2: Net-(D_SHIFT-Pad2) -> (no net)
- K_SHIFT1 pad 1: /col12 -> (no net)
- K_SHIFT1 pad 2: Net-(D_SHIFT1-Pad2) -> (no net)
- K_SLASH pad 1: /col11 -> (no net)
- K_SLASH pad 2: Net-(D_SLASH-Pad2) -> (no net)
- K_SPACE pad 1: /col14 -> (no net)
- K_SPACE pad 2: Net-(D_SPACE-Pad2) -> (no net)
- K_SPACE1 pad 1: /col14 -> (no net)
- K_SPACE1 pad 2: Net-(D_SPACE1-Pad2) -> (no net)
- K_SPACE2 pad 1: /col6 -> (no net)
- K_SPACE2 pad 2: Net-(D_SPACE2-Pad2) -> (no net)
- K_T pad 1: /col6 -> (no net)
- K_T pad 2: Net-(D_T-Pad2) -> (no net)
- K_TAB pad 1: /col0 -> (no net)
- K_TAB pad 2: Net-(D_TAB-Pad2) -> (no net)
- K_U pad 1: /col8 -> (no net)
- K_U pad 2: Net-(D_U-Pad2) -> (no net)
- K_V pad 1: /col5 -> (no net)
- K_V pad 2: Net-(D_V-Pad2) -> (no net)
- K_W pad 1: /col3 -> (no net)
- K_W pad 2: Net-(D_W-Pad2) -> (no net)
- K_WIN pad 1: /col1 -> (no net)
- K_WIN pad 2: Net-(D_WIN-Pad2) -> (no net)
- K_WIN1 pad 1: /col11 -> (no net)
- K_WIN1 pad 2: Net-(D_WIN1-Pad2) -> (no net)
- K_X pad 1: /col3 -> (no net)
- K_X pad 2: Net-(D_X-Pad2) -> (no net)
- K_Y pad 1: /col7 -> (no net)
- K_Y pad 2: Net-(D_Y-Pad2) -> (no net)
- K_Z pad 1: /col2 -> (no net)
- K_Z pad 2: Net-(D_Z-Pad2) -> (no net)
- K_` pad 1: /col0 -> (no net)
- K_` pad 2: Net-(D_`-Pad2) -> (no net)
Routing:
- net (no net): track 609.2 -> 2172.6 mm, vias 10 -> 19
- net GND: track 29.8 -> 134.1 mm, vias 6 -> 13
- added copper zone on F.Cu, net (none)
- removed copper zone on F.Cu, net VCC
