File: LED projects/Led Flashlight/Led Flashlight.kicad_pcb (KiCad board)
At the start: 2 copper layers, 41.3 x 26.5 mm, 37 parts

Commit message: update
Parts:
- added REF**: DIP794W45P254L1969H508Q14, CD4047BE:DIP794W45P254L1969H508Q14, B.Cu at (116.8, 102.3)
- moved REF** 20.4 mm to (129.9, 99.3)
- moved REF** 6.21 mm to (99.5, 105.8)
- moved REF** 6.21 mm to (134.1, 105.9)
Routing:
- net (no net): track 163.1 -> 177.7 mm
Other:
- board size 41.3 x 26.5 mm -> 40.9 x 32.8 mm
Changed lines of the file:
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@@
   (net 0 "")
   (footprint "MountingHole:MountingHole_2.2mm_M2" (layer "F.Cu")
-    (at 99.52 99.55)
+    (at 99.5 105.76)
     (descr "Mounting Hole 2.2mm, no annular, M2")
     (tags "mounting hole 2.2mm no annular m2")
@@
   )
   (footprint "MountingHole:MountingHole_2.2mm_M2" (layer "F.Cu")
-    (at 134.16 99.65)
+    (at 134.14 105.86)
     (descr "Mounting Hole 2.2mm, no annular, M2")
     (tags "mounting hole 2.2mm no annular m2")
@@
   )
   (footprint "Connector_PinHeader_2.00mm:PinHeader_1x01_P2.00mm_Vertical" (layer "F.Cu")
-    (at 129.08 78.97)
+    (at 129.87 99.33)
     (descr "Through hole straight pin header, 1x01, 2.00mm pitch, single row")
     (tags "Through hole pin header THT 1x01 2.00mm single row")
@@
     )
   )
+  (footprint "CD4047BE:DIP794W45P254L1969H508Q14" (layer "B.Cu")
+    (at 116.76 102.32 -90)
+    (attr through_hole)
+    (fp_text reference "REF**" (at -0.825 11.135 90) (layer "B.SilkS") hide
+        (effects (font (size 1 1) (thickness 0.15)) (justify mirror))
+    )
+    (fp_text value "DIP794W45P254L1969H508Q14" (at 11.875 -11.135 90) (layer "B.Fab") hide
+        (effects (font (size 1 1) (thickness 0.15)) (justify mirror))
+    )
+    (fp_line (start -3.3 -9.845) (end -3.3 -8.525)
+      (stroke (width 0.127) (type solid)) (layer "B.SilkS"))
+    (fp_line (start -3.3 8.525) (end -3.3 9.845)
+      (stroke (width 0.127) (type solid)) (layer "B.SilkS"))
+    (fp_line (start -3.3 9.845) (end 3.3 9.845)
+      (stroke (width 0.127) (type solid)) (layer "B.SilkS"))
+    (fp_line (start 3.3 -9.845) (end -3.3 -9.845)
+      (stroke (width 0.127) (type solid)) (layer "B.SilkS"))
+    (fp_line (start 3.3 -8.525) (end 3.3 -9.845)
+      (stroke (width 0.127) (type solid)) (layer "B.SilkS"))
+    (fp_line (start 3.3 9.845) (end 3.3 8.525)
+      (stroke (width 0.127) (type solid)) (layer "B.SilkS"))
+    (fp_circle (center -5.055 7.62) (end -4.955 7.62)
+      (stroke (width 0.2) (type solid)) (fill none) (layer "B.SilkS"))
+    (fp_line (start -4.805 10.095) (end -4.805 -10.095)
+      (stroke (width 0.05) (type solid)) (layer "B.CrtYd"))
+    (fp_line (start 4.805 -10.095) (end -4.805 -10.095)
+      (stroke (width 0.05) (type solid)) (layer "B.CrtYd"))
+    (fp_line (start 4.805 10.095) (end -4.805 10.095)
+      (stroke (width 0.05) (type solid)) (layer "B.CrtYd"))
+    (fp_line (start 4.805 10.095) (end 4.805 -10.095)
+      (stroke (width 0.05) (type solid)) (layer "B.CrtYd"))
+    (fp_line (start -3.3 -9.845) (end 3.3 -9.845)
+      (stroke (width 0.127) (type solid)) (layer "B.Fab"))
+    (fp_line (start -3.3 9.845) (end -3.3 -9.845)
+      (stroke (width 0.127) (type solid)) (layer "B.Fab"))
+    (fp_line (start -3.3 9.845) (end 3.3 9.845)
+      (stroke (width 0.127) (type solid)) (layer "B.Fab"))
+    (fp_line (start 3.3 9.845) (end 3.3 -9.845)
+      (stroke (width 0.127) (type solid)) (layer "B.Fab"))
+    (fp_circle (center -5.055 7.62) (end -4.955 7.62)
+      (stroke (width 0.2) (type solid)) (fill none) (layer "B.Fab"))
+    (pad "1" thru_hole rect (at -3.97 7.62 270) (size 1.17 1.17) (drill 0.77) (layers "*.Cu" "*.Mask")
+      (solder_mask_margin 0.102))
+    (pad "2" thru_hole circle (at -3.97 5.08 270) (size 1.17 1.17) (drill 0.77) (layers "*.Cu" "*.Mask")
+      (solder_mask_margin 0.102))
+    (pad "3" thru_hole circle (at -3.97 2.54 270) (size 1.17 1.17) (drill 0.77) (layers "*.Cu" "*.Mask")
+      (solder_mask_margin 0.102))
+    (pad "4" thru_hole circle (at -3.97 0 270) (size 1.17 1.17) (drill 0.77) (layers "*.Cu" "*.Mask")
+      (solder_mask_margin 0.102))
+    (pad "5" thru_hole circle (at -3.97 -2.54 270) (size 1.17 1.17) (drill 0.77) (layers "*.Cu" "*.Mask")
+      (solder_mask_margin 0.102))
+    (pad "6" thru_hole circle (at -3.97 -5.08 270) (size 1.17 1.17) (drill 0.77) (layers "*.Cu" "*.Mask")
+      (solder_mask_margin 0.102))
+    (pad "7" thru_hole circle (at -3.97 -7.62 270) (size 1.17 1.17) (drill 0.77) (layers "*.Cu" "*.Mask")
+      (solder_mask_margin 0.102))
+    (pad "8" thru_hole circle (at 3.97 -7.62 270) (size 1.17 1.17) (drill 0.77) (layers "*.Cu" "*.Mask")
+      (solder_mask_margin 0.102))
+    (pad "9" thru_hole circle (at 3.97 -5.08 270) (size 1.17 1.17) (drill 0.77) (layers "*.Cu" "*.Mask")
+      (solder_mask_margin 0.102))
+    (pad "10" thru_hole circle (at 3.97 -2.54 270) (size 1.17 1.17) (drill 0.77) (layers "*.Cu" "*.Mask")
+      (solder_mask_margin 0.102))
+    (pad "11" thru_hole circle (at 3.97 0 270) (size 1.17 1.17) (drill 0.77) (layers "*.Cu" "*.Mask")
+      (solder_mask_margin 0.102))
+    (pad "12" thru_hole circle (at 3.97 2.54 270) (size 1.17 1.17) (drill 0.77) (layers "*.Cu" "*.Mask")
+      (solder_mask_margin 0.102))
+    (pad "13" thru_hole circle (at 3.97 5.08 270) (size 1.17 1.17) (drill 0.77) (layers "*.Cu" "*.Mask")
+      (solder_mask_margin 0.102))
+    (pad "14" thru_hole circle (at 3.97 7.62 270) (size 1.17 1.17) (drill 0.77) (layers "*.Cu" "*.Mask")
+      (solder_mask_margin 0.102))
+  )
   (footprint "Resistor_SMD:R_0805_2012Metric" (layer "B.Cu")
     (at 108.6525 94.03 180)
@@
     )
   )
-  (gr_arc (start 137.32 99.72) (mid 136.44132 101.84132) (end 134.32 102.72)
+  (gr_line (start 96.25 105.96) (end 96.25 79.19)
     (stroke (width 0.1) (type default)) (layer "Edge.Cuts"))
-  (gr_line (start 96.01 99.72) (end 96.01 79.18)
+  (gr_line (start 99.25 76.19) (end 134.12 76.19)
     (stroke (width 0.1) (type default)) (layer "Edge.Cuts"))
-  (gr_line (start 137.32 79.18) (end 137.32 99.72)
+  (gr_line (start 137.12 79.19) (end 137.12 105.96)
     (stroke (width 0.1) (type default)) (layer "Edge.Cuts"))
-  (gr_arc (start 99.01 102.72) (mid 96.88868 101.84132) (end 96.01 99.72)
+  (gr_arc (start 134.12 76.19) (mid 136.24132 77.06868) (end 137.12 79.19)
     (stroke (width 0.1) (type default)) (layer "Edge.Cuts"))
-  (gr_arc (start 134.32 76.18) (mid 136.44132 77.05868) (end 137.32 79.18)
+  (gr_arc (start 99.25 108.96) (mid 97.12868 108.08132) (end 96.25 105.96)
     (stroke (width 0.1) (type default)) (layer "Edge.Cuts"))
-  (gr_line (start 99.01 76.18) (end 134.32 76.18)
+  (gr_arc (start 137.12 105.96) (mid 136.24132 108.08132) (end 134.12 108.96)
     (stroke (width 0.1) (type default)) (layer "Edge.Cuts"))
-  (gr_line (start 134.32 102.72) (end 99.01 102.72)
+  (gr_line (start 134.12 108.96) (end 99.25 108.96)
     (stroke (width 0.1) (type default)) (layer "Edge.Cuts"))
-  (gr_arc (start 96.01 79.18) (mid 96.88868 77.05868) (end 99.01 76.18)
+  (gr_arc (start 96.25 79.19) (mid 97.12868 77.06868) (end 99.25 76.19)
     (stroke (width 0.1) (type default)) (layer "Edge.Cuts"))
   (segment (start 123.07 93.75) (end 123.26 93.56) (width 0.25) (layer "F.Cu") (net 0))
@@
   (segment (start 123.05 87.1) (end 123.05 85.46) (width 0.25) (layer "F.Cu") (net 0))
   (segment (start 117.36 89.31) (end 117.32 89.27) (width 0.25) (layer "F.Cu") (net 0))
+  (segment (start 129.87 99.33) (end 131.42 99.33) (width 0.25) (layer "F.Cu") (net 0))
   (segment (start 130.93 82.95) (end 130.99 82.95) (width 0.25) (layer "F.Cu") (net 0))
   (segment (start 123.05 85.46) (end 123.36 85.15) (width 0.25) (layer "F.Cu") (net 0))
   (segment (start 101.85 96.99) (end 104.41 99.55) (width 0.25) (layer "F.Cu") (net 0))
   (segment (start 107.55 95.45) (end 107.55 93.81) (width 0.25) (layer "F.Cu") (net 0))
+  (segment (start 132.99 84.82) (end 131.16 82.99) (width 0.25) (layer "F.Cu") (net 0))
   (segment (start 101.65 82.96) (end 101.64 82.95) (width 0.25) (layer "F.Cu") (net 0))
   (segment (start 107.52 80.4) (end 107.73 80.19) (width 0.25) (layer "F.Cu") (net 0))
-  (segment (start 129.08 79.13) (end 131.03 81.08) (width 0.25) (layer "F.Cu") (net 0))
   (segment (start 125.26 95.44) (end 125.26 93.59) (width 0.25) (layer "F.Cu") (net 0))
   (segment (start 107.53 87.11) (end 107.53 85.25) (width 0.25) (layer "F.Cu") (net 0))
@@
   (segment (start 107.53 85.25) (end 107.7 85.08) (width 0.25) (layer "F.Cu") (net 0))
   (segment (start 109.74 93.71) (end 109.72 93.69) (width 0.25) (layer "F.Cu") (net 0))
+  (segment (start 131.42 99.33) (end 132.99 97.76) (width 0.25) (layer "F.Cu") (net 0))
   (segment (start 115.44 93.63) (end 115.4 93.59) (width 0.25) (layer "F.Cu") (net 0))
   (segment (start 109.71 80.31) (end 109.59 80.19) (width 0) (layer "F.Cu") (net 0))
@@
   (segment (start 101.83 87.32) (end 101.88 87.37) (width 0.25) (layer "F.Cu") (net 0))
   (segment (start 115.42 85.16) (end 115.46 85.12) (width 0.25) (layer "F.Cu") (net 0))
-  (segment (start 129.08 78.97) (end 129.08 79.13) (width 0.25) (layer "F.Cu") (net 0))
   (segment (start 109.71 82.96) (end 109.71 80.31) (width 0.25) (layer "F.Cu") (net 0))
+  (segment (start 132.99 97.76) (end 132.99 84.82) (width 0.25) (layer "F.Cu") (net 0))
+  (segment (start 131.16 82.99) (end 131.03 82.99) (width 0.25) (layer "F.Cu") (net 0))
   (segment (start 107.55 93.81) (end 107.67 93.69) (width 0.25) (layer "F.Cu") (net 0))
   (segment (start 115.41 82.96) (end 115.41 80.35) (width 0.25) (layer "F.Cu") (net 0))
@@
   (segment (start 115.44 95.45) (end 115.44 93.63) (width 0.25) (layer "F.Cu") (net 0))
   (segment (start 101.84 91.3) (end 101.84 91.56) (width 0.25) (layer "F.Cu") (net 0))
-  (segment (start 131.03 82.99) (end 131.03 81.08) (width 0.25) (layer "F.Cu") (net 0))
   (segment (start 115.43 89.37) (end 115.56 89.24) (width 0.25) (layer "F.Cu") (net 0))
   (segment (start 115.41 80.35) (end 115.5 80.26) (width 0) (layer "F.Cu") (net 0))
@@
         (xy 93.21 73.86)
         (xy 137.87 73.71)
-        (xy 137.8 105.46)
-        (xy 93.29 105.53)
+        (xy 137.85 109.37)
+        (xy 93.34 109.44)
         (xy 93.21 73.79)
       )
@@
         (xy 93.21 73.79)
         (xy 137.87 73.71)
-        (xy 137.8 105.46)
-        (xy 93.29 105.53)
+        (xy 137.95 109.37)
+        (xy 93.44 109.44)
       )
     )
