File: LED projects/LED flashlight 2/PCB/LED2/LED2.kicad_pcb (KiCad board)
At the start: 2 copper layers, 21 x 12.5 mm, 5 parts, among them SW1 SW_Push

Commit message: led2 update
Parts:
- BT1: footprint Connector_PinHeader_1.27mm:PinHeader_1x02_P1.27mm_Vertical -> Connector_PinHeader_2.54mm:PinHeader_1x02_P2.54mm_Vertical
- moved BatteryChargeModule1 14.1 mm to (156.1, 98.8)
- moved D1 14.1 mm to (143.6, 98.0)
- moved R1 14.1 mm to (147.6, 103.4)
- moved SW1 14.1 mm to (152.1, 99.3)
- moved BT1 13.8 mm to (159.7, 97.8)

Commit message: update
Parts:
- added R1: R_US, Resistor_THT:R_Axial_DIN0207_L6.3mm_D2.5mm_P7.62mm_Horizontal, F.Cu at (152.1, 103.1)
Routing:
- net Net-(R1-Pad2): track 5.25 -> 7.36 mm
- net Net-(BatteryChargeModule1--): track 4.31 -> 6.42 mm
