File: LED projects/LED flashlight 3/LED flashlight/LED flashlight.kicad_pcb (KiCad board)
At the start: 2 copper layers, 37.1 x 17.5 mm, 14 parts, among them P1 USB_C_Plug_USB2.0, SW1 SW_Push, U1 TP4056

Commit message: update
Parts:
- moved P1 0.73 mm to (126.1, 91.5)
Routing:
- net Earth: track 58.1 -> 52.3 mm, vias 6 -> 4
- net Net-(P1-VBUS-PadA4): track 16.0 -> 14.8 mm, vias 0 -> 1
- net unconnected-(P1-SHIELD-PadS1): vias 0 -> 1
Changed lines of the file:
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@@
 		(tags "LED")
 		(property "Reference" "D4"
-			(at -0.08 -0.21 360)
+			(at -0.08 -0.21 0)
 			(layer "F.SilkS")
 			(effects
@@
 		)
 		(property "Value" "LED"
-			(at 0 1.82 360)
+			(at 0 1.82 0)
 			(layer "F.Fab")
 			(hide yes)
@@
 		(tags "resistor")
 		(property "Reference" "R5"
-			(at 0.045 0.045 360)
+			(at 0.045 0.045 0)
 			(layer "F.SilkS")
 			(effects
@@
 		(tags "capacitor")
 		(property "Reference" "D1"
-			(at -0.09 -0.02 360)
+			(at -0.09 -0.02 0)
 			(layer "F.SilkS")
 			(effects
@@
 		)
 		(property "Value" "D_Capacitance"
-			(at 0 1.85 360)
+			(at 0 1.85 0)
 			(layer "F.Fab")
 			(hide yes)
@@
 	(footprint "Connector_USB:USB_C_Receptacle_GCT_USB4105-xx-A_16P_TopMnt_Horizontal"
 		(layer "F.Cu")
-		(at 126 92.27 -90)
+		(at 126.062221 91.539014 -90)
 		(descr "USB 2.0 Type C Receptacle, GCT, 16P, top mounted, horizontal, 5A: https://gct.co/files/drawings/usb4105.pdf")
 		(tags "USB C Type-C Receptacle SMD USB 2.0 16P 16C USB4105-15-A USB4105-15-A-060 USB4105-15-A-120 USB4105-GF-A USB4105-GF-A-060 USB4105-GF-A-120")
@@
 		(tags "LED")
 		(property "Reference" "D5"
-			(at 0.03 -0.07 360)
+			(at 0.03 -0.07 0)
 			(layer "F.SilkS")
 			(effects
@@
 		)
 		(property "Value" "LED"
-			(at 0 1.82 360)
+			(at 0 1.82 0)
 			(layer "F.Fab")
 			(hide yes)
@@
 		(at 141.935 94.985)
 		(property "Reference" "U1"
-			(at 3.005 3.295 360)
+			(at 3.005 3.295 0)
 			(layer "F.SilkS")
 			(effects
@@
 		)
 		(property "Value" "TP4056"
-			(at 6.825 3.362 360)
+			(at 6.825 3.362 0)
 			(layer "F.Fab")
 			(hide yes)
@@
 		)
 		(property "Footprint" "Personal:SOP127P600X175-9N"
-			(at 0 0 360)
+			(at 0 0 0)
 			(layer "F.Fab")
 			(hide yes)
@@
 		)
 		(property "Datasheet" ""
-			(at 0 0 360)
+			(at 0 0 0)
 			(layer "F.Fab")
 			(hide yes)
@@
 		)
 		(property "Description" ""
-			(at 0 0 360)
+			(at 0 0 0)
 			(layer "F.Fab")
 			(hide yes)
@@
 		(tags "resistor")
 		(property "Reference" "R4"
-			(at 0 -0.1 360)
+			(at 0 -0.1 0)
 			(layer "F.SilkS")
 			(effects
@@
 		)
 		(property "Value" "R"
-			(at 0 1.82 360)
+			(at 0 1.82 0)
 			(layer "F.Fab")
 			(hide yes)
@@
 	)
 	(segment
-		(start 130.245 95.99)
-		(end 129.725 95.47)
-		(width 0.2)
-		(layer "F.Cu")
-		(net 1)
-	)
-	(segment
-		(start 131.9475 95.99)
-		(end 130.245 95.99)
+		(start 131.985 93.05)
+		(end 132.085 93.15)
 		(width 0.2)
 		(layer "F.Cu")
@@
 	)
 	(segment
-		(start 131.985 93.05)
-		(end 132.085 93.15)
+		(start 139.46 93.06)
+		(end 139.43 93.03)
 		(width 0.2)
 		(layer "F.Cu")
@@
 	)
 	(segment
-		(start 139.46 93.06)
-		(end 139.43 93.03)
+		(start 129.742221 94.739014)
+		(end 130.696514 94.739014)
 		(width 0.2)
 		(layer "F.Cu")
@@
 	)
 	(segment
-		(start 129.725 89.07)
-		(end 131.265 89.07)
+		(start 130.534014 88.339014)
+		(end 131.985 89.79)
 		(width 0.2)
 		(layer "F.Cu")
@@
 	)
 	(segment
-		(start 154.82 98.265)
-		(end 154.82 99.18)
+		(start 129.742221 88.339014)
+		(end 130.534014 88.339014)
 		(width 0.2)
 		(layer "F.Cu")
@@
 	)
 	(segment
-		(start 131.265 89.07)
-		(end 131.985 89.79)
+		(start 154.82 98.265)
+		(end 154.82 99.18)
 		(width 0.2)
 		(layer "F.Cu")
@@
 		(net 1)
 	)
-	(via
-		(at 129.725 95.47)
-		(size 0.6)
-		(drill 0.3)
-		(layers "F.Cu" "B.Cu")
-		(net 1)
-	)
-	(via
-		(at 129.725 89.07)
-		(size 0.6)
-		(drill 0.3)
-		(layers "F.Cu" "B.Cu")
+	(segment
+		(start 130.696514 94.739014)
+		(end 131.9475 95.99)
+		(width 0.2)
+		(layer "F.Cu")
 		(net 1)
 	)
@@
 	)
 	(segment
-		(start 129.725 89.07)
-		(end 129.725 95.47)
-		(width 0.2)
-		(layer "B.Cu")
-		(net 1)
-	)
-	(segment
 		(start 149.52 94.46)
 		(end 146.1 97.88)
@@
 	)
 	(segment
-		(start 128.82 94.485)
-		(end 128.38 94.045)
+		(start 128.113267 89.572026)
+		(end 127.687128 89.145887)
 		(width 0.2)
 		(layer "F.Cu")
@@
 	)
 	(segment
-		(start 131.5075 86.39)
-		(end 127.85 86.39)
+		(start 129.192362 89.139014)
+		(end 128.75935 89.572026)
 		(width 0.2)
 		(layer "F.Cu")
@@
 	)
 	(segment
-		(start 129.725 94.67)
-		(end 129.54 94.485)
+		(start 127.687128 89.145887)
+		(end 127.687128 86.850231)
 		(width 0.2)
 		(layer "F.Cu")
@@
 	)
 	(segment
-		(start 128.38 90.07)
-		(end 129.525 90.07)
+		(start 128.73873 93.484954)
+		(end 128.73873 89.592646)
 		(width 0.2)
 		(layer "F.Cu")
@@
 	)
 	(segment
-		(start 127.85 86.39)
-		(end 127.09 87.15)
+		(start 129.742221 93.939014)
+		(end 129.19279 93.939014)
 		(width 0.2)
 		(layer "F.Cu")
@@
 	)
 	(segment
-		(start 129.525 90.07)
-		(end 129.725 89.87)
+		(start 131.153254 86.035754)
+		(end 132.0075 86.89)
 		(width 0.2)
 		(layer "F.Cu")
@@
 	)
 	(segment
-		(start 128.38 94.045)
-		(end 128.38 90.07)
+		(start 128.75935 89.572026)
+		(end 128.113267 89.572026)
 		(width 0.2)
 		(layer "F.Cu")
@@
 	)
 	(segment
-		(start 127.09 88.98)
-		(end 128.18 90.07)
+		(start 127.687128 86.850231)
+		(end 128.501605 86.035754)
 		(width 0.2)
 		(layer "F.Cu")
@@
 	)
 	(segment
-		(start 127.09 87.15)
-		(end 127.09 88.98)
+		(start 129.742221 89.139014)
+		(end 129.192362 89.139014)
 		(width 0.2)
 		(layer "F.Cu")
@@
 	)
 	(segment
-		(start 132.0075 86.89)
-		(end 131.5075 86.39)
+		(start 129.19279 93.939014)
+		(end 128.73873 93.484954)
 		(width 0.2)
 		(layer "F.Cu")
@@
 	)
 	(segment
-		(start 129.54 94.485)
-		(end 128.82 94.485)
+		(start 128.501605 86.035754)
+		(end 131.153254 86.035754)
 		(width 0.2)
 		(layer "F.Cu")
@@
 	)
 	(segment
-		(start 128.18 90.07)
-		(end 128.38 90.07)
+		(start 128.73873 89.592646)
+		(end 128.75935 89.572026)
 		(width 0.2)
 		(layer "F.Cu")
 		(net 6)
 	)
+	(via
+		(at 129.725 89.07)
+		(size 0.6)
+		(drill 0.3)
+		(layers "F.Cu" "B.Cu")
+		(net 6)
+	)
+	(via
+		(at 129.725 95.47)
+		(size 0.6)
+		(drill 0.3)
+		(layers "F.Cu" "B.Cu")
+		(net 9)
+	)
 	(segment

Commit message: update
Parts:
- removed D3: LED, LED_THT:LED_D5.0mm_Horizontal_O1.27mm_Z3.0mm
- added LED: Battery, Connector_PinHeader_2.54mm:PinHeader_1x02_P2.54mm_Vertical, F.Cu at (159.7, 88.3)
