File: LED projects/LED flashlight 3/LED flashlight/LED flashlight.kicad_pcb (KiCad board)
At the start: 2 copper layers, 37.1 x 17.5 mm, 14 parts, among them P1 USB_C_Plug_USB2.0, SW1 SW_Push, U1 TP4056

Commit message: update
Parts:
- added R6: R, Resistor_SMD:R_1206_3216Metric, F.Cu at (133.4, 98.5)
- added R7: R, Resistor_SMD:R_1206_3216Metric, F.Cu at (133.5, 84.6)
Routing:
- net unconnected-(P1-SHIELD-PadS1): track 0.00 -> 17.0 mm
- net Earth: track 52.3 -> 63.4 mm
- net unconnected-(P1-CC-PadA5): track 0.00 -> 7.20 mm, vias 0 -> 2
- net unconnected-(P1-VCONN-PadB5): track 0.00 -> 6.77 mm, vias 0 -> 2
- added copper zone on B.Cu, net Earth
- added copper zone on F.Cu, net Earth
- removed copper zone on B.Cu, net (none)
- removed copper zone on F.Cu, net (none)
